File: sch/Display.sch (KiCad schematic (older format))
At the start: 1 part

Commit message: cambios sch
Parts:
- removed U?: DE113-XX-XX, Display_7Segment:DE113-XX-XX, symbol Display_Character:DE113-XX-XX
Changed lines of the file:
@@
 $Descr A4 11693 8268
 encoding utf-8
-Sheet 9 9
+Sheet 8 9
 Title ""
 Date ""
@@
 Comment4 ""
 $EndDescr
-$Comp
-L Display_Character:DE113-XX-XX U?
-U 1 1 5B7842F9
-P 6150 2750
-F 0 "U?" H 6150 4017 50  0000 C CNN
-F 1 "DE113-XX-XX" H 6150 3926 50  0000 C CNN
-F 2 "Display_7Segment:DE113-XX-XX" H 6150 1450 50  0001 C CNN
-F 3 "http://www.display-elektronik.de/filter/DE113-MS-20_75.pdf" H 5950 2950 50  0001 C CNN
-	1    6150 2750
-	1    0    0    -1
-$EndComp
 $EndSCHEMATC
