File: sch/LPC.sch (KiCad schematic (older format))
At the start: 1 part

Commit message: cambios sch
Connections:
- net labels added: CAP2.1, CTS1, RTS1, RXD1, TXD1
- net labels removed: RXD2, TXD2
- wire segments 17 -> 20
- no-connect marks 53 -> 50
Changed lines of the file:
@@
 $Descr A4 11693 8268
 encoding utf-8
-Sheet 4 9
+Sheet 9 9
 Title ""
 Date ""
@@
 Wire Wire Line
 	3950 3800 3600 3800
-Text HLabel 6850 2600 2    50   Input ~ 0
-RXD2
-Text HLabel 6850 2500 2    50   Output ~ 0
-TXD2
-Wire Wire Line
-	6350 2500 6850 2500
-Wire Wire Line
-	6850 2600 6350 2600
 Wire Wire Line
 	3950 2000 3650 2000
@@
 NoConn ~ 6350 3600
 NoConn ~ 6350 3500
-NoConn ~ 6350 3400
 NoConn ~ 6350 3300
 NoConn ~ 6350 3200
 NoConn ~ 6350 3100
 NoConn ~ 6350 3000
-NoConn ~ 6350 2900
-NoConn ~ 6350 2800
-NoConn ~ 6350 2700
-NoConn ~ 6350 2400
 NoConn ~ 6350 2300
 NoConn ~ 6350 2200
@@
 Wire Wire Line
 	3650 2300 3950 2300
+Wire Wire Line
+	6350 2400 6850 2400
+Text HLabel 6850 2400 2    50   Input ~ 0
+CAP2.1
+NoConn ~ 6350 2500
+NoConn ~ 6350 2600
+Wire Wire Line
+	6350 2700 6850 2700
+Wire Wire Line
+	6350 2800 6850 2800
+Wire Wire Line
+	6350 2900 6850 2900
+Wire Wire Line
+	6350 3400 6850 3400
+Text HLabel 6850 2700 2    50   Output ~ 0
+TXD1
+Text HLabel 6850 2800 2    50   Input ~ 0
+RXD1
+Text HLabel 6850 2900 2    50   Input ~ 0
+CTS1
+Text HLabel 6850 3400 2    50   Output ~ 0
+RTS1
 $EndSCHEMATC
