File: sch/ZigBee.sch (KiCad schematic (older format))
At the start: 1 part

Commit message: cambios sch
Connections:
- net labels added: RSSI, RTS
- wire segments 14 -> 20
- no-connect marks 10 -> 8
Changed lines of the file:
@@
 $Descr A4 11693 8268
 encoding utf-8
-Sheet 5 9
+Sheet 4 9
 Title ""
 Date ""
@@
 L power:+3.3V #PWR?
 U 1 1 5B71F637
-P 6100 2850
-F 0 "#PWR?" H 6100 2700 50  0001 C CNN
-F 1 "+3.3V" H 6115 3023 50  0000 C CNN
-F 2 "" H 6100 2850 50  0001 C CNN
-F 3 "" H 6100 2850 50  0001 C CNN
-	1    6100 2850
+P 6050 2800
+F 0 "#PWR?" H 6050 2650 50  0001 C CNN
+F 1 "+3.3V" H 6065 2973 50  0000 C CNN
+F 2 "" H 6050 2800 50  0001 C CNN
+F 3 "" H 6050 2800 50  0001 C CNN
+	1    6050 2800
 	1    0    0    -1
 $EndComp
 Wire Wire Line
-	6100 2950 6100 2850
+	6050 2900 6050 2800
 $Comp
 L power:GND #PWR?
 U 1 1 5B71F679
-P 6000 4250
-F 0 "#PWR?" H 6000 4000 50  0001 C CNN
-F 1 "GND" H 6005 4077 50  0000 C CNN
-F 2 "" H 6000 4250 50  0001 C CNN
-F 3 "" H 6000 4250 50  0001 C CNN
-	1    6000 4250
+P 5950 4200
+F 0 "#PWR?" H 5950 3950 50  0001 C CNN
+F 1 "GND" H 5955 4027 50  0000 C CNN
+F 2 "" H 5950 4200 50  0001 C CNN
+F 3 "" H 5950 4200 50  0001 C CNN
+	1    5950 4200
 	1    0    0    -1
 $EndComp
 Wire Wire Line
-	6000 4250 6000 4150
-NoConn ~ 6800 3850
-NoConn ~ 6800 3950
-NoConn ~ 6800 3550
-NoConn ~ 6800 3450
-NoConn ~ 6800 3350
-NoConn ~ 6800 3250
-NoConn ~ 5400 3950
-NoConn ~ 5400 3850
-NoConn ~ 5400 3750
-NoConn ~ 5400 3650
-Text HLabel 8150 3250 2    50   Input ~ 0
+	5950 4200 5950 4100
+NoConn ~ 6750 3800
+NoConn ~ 6750 3500
+NoConn ~ 6750 3400
+NoConn ~ 6750 3200
+NoConn ~ 5350 3900
+NoConn ~ 5350 3800
+NoConn ~ 5350 3700
+NoConn ~ 5350 3600
+Text HLabel 8100 3200 2    50   Input ~ 0
 TXD2
-Text HLabel 8150 3150 2    50   Output ~ 0
+Text HLabel 8100 3100 2    50   Output ~ 0
 RXD2
 $Comp
 L dk_RF-Transceiver-Modules:XB24CZ7PIT-004 MOD?
 U 1 1 5B734775
-P 6200 3750
-F 0 "MOD?" H 5600 4500 60  0000 C CNN
-F 1 "XB24CZ7PIT-004" H 6300 4500 60  0000 C CNN
-F 2 "digikey-footprints:XBEE-20_THT" H 6400 3950 60  0001 L CNN
-F 3 "https://www.digi.com/resources/documentation/digidocs/pdfs/90001500.pdf" H 6400 4050 60  0001 L CNN
-F 4 "602-1557-ND" H 6400 4150 60  0001 L CNN "Digi-Key_PN"
-F 5 "XB24CZ7PIT-004" H 6400 4250 60  0001 L CNN "MPN"
-F 6 "RF/IF and RFID" H 6400 4350 60  0001 L CNN "Category"
-F 7 "RF Transceiver Modules" H 6400 4450 60  0001 L CNN "Family"
-F 8 "https://www.digi.com/resources/documentation/digidocs/pdfs/90001500.pdf" H 6400 4550 60  0001 L CNN "DK_Datasheet_Link"
-F 9 "/product-detail/en/digi-international/XB24CZ7PIT-004/602-1557-ND/5322371" H 6400 4650 60  0001 L CNN "DK_Detail_Page"
-F 10 "RF TXRX MOD 802.15.4 TRACE ANT" H 6400 4750 60  0001 L CNN "Description"
-F 11 "Digi International" H 6400 4850 60  0001 L CNN "Manufacturer"
-F 12 "Active" H 6400 4950 60  0001 L CNN "Status"
-	1    6200 3750
+P 6150 3700
+F 0 "MOD?" H 5550 4450 60  0000 C CNN
+F 1 "XB24CZ7PIT-004" H 6250 4450 60  0000 C CNN
+F 2 "digikey-footprints:XBEE-20_THT" H 6350 3900 60  0001 L CNN
+F 3 "https://www.digi.com/resources/documentation/digidocs/pdfs/90001500.pdf" H 6350 4000 60  0001 L CNN
+F 4 "602-1557-ND" H 6350 4100 60  0001 L CNN "Digi-Key_PN"
+F 5 "XB24CZ7PIT-004" H 6350 4200 60  0001 L CNN "MPN"
+F 6 "RF/IF and RFID" H 6350 4300 60  0001 L CNN "Category"
+F 7 "RF Transceiver Modules" H 6350 4400 60  0001 L CNN "Family"
+F 8 "https://www.digi.com/resources/documentation/digidocs/pdfs/90001500.pdf" H 6350 4500 60  0001 L CNN "DK_Datasheet_Link"
+F 9 "/product-detail/en/digi-international/XB24CZ7PIT-004/602-1557-ND/5322371" H 6350 4600 60  0001 L CNN "DK_Detail_Page"
+F 10 "RF TXRX MOD 802.15.4 TRACE ANT" H 6350 4700 60  0001 L CNN "Description"
+F 11 "Digi International" H 6350 4800 60  0001 L CNN "Manufacturer"
+F 12 "Active" H 6350 4900 60  0001 L CNN "Status"
+	1    6150 3700
 	1    0    0    -1
 $EndComp
 Wire Wire Line
-	5400 3250 4700 3250
+	5000 3200 5000 3100
 Wire Wire Line
-	4700 3250 4700 3150
-Wire Wire Line
-	5150 3150 5400 3150
-Text Label 5150 3150 0    50   ~ 0
+	5100 3100 5350 3100
+Text Label 5100 3100 0    50   ~ 0
 TXD1
-Text Label 7050 3150 2    50   ~ 0
+Text Label 7100 3100 2    50   ~ 0
 RXD2
-Wire Wire Line
-	7050 3150 6800 3150
-Text Label 5050 3450 0    50   ~ 0
+Text Label 5000 3400 0    50   ~ 0
 SleepRQ
 Wire Wire Line
-	5050 3450 5400 3450
+	5000 3400 5350 3400
 Wire Wire Line
-	6800 3750 7150 3750
+	6750 3700 7100 3700
 Wire Wire Line
-	6800 3650 7150 3650
-Text Label 7150 3650 2    50   ~ 0
+	6750 3600 7100 3600
+Text Label 7100 3600 2    50   ~ 0
 CTS
-Text Label 7150 3750 2    50   ~ 0
+Text Label 7100 3700 2    50   ~ 0
 SLEEP
-Text HLabel 8150 3350 2    50   Input ~ 0
+Text HLabel 8100 3300 2    50   Input ~ 0
 SLRQ
-Text HLabel 8150 3450 2    50   Output ~ 0
+Text HLabel 8100 3400 2    50   Output ~ 0
 SLEEP
-Text HLabel 8150 3550 2    50   Output ~ 0
+Text HLabel 8100 3500 2    50   Output ~ 0
 CTS
 Wire Wire Line
-	8150 3150 7600 3150
+	8100 3100 7550 3100
 Wire Wire Line
-	8150 3250 7600 3250
+	8100 3200 7550 3200
 Wire Wire Line
-	7600 3350 8150 3350
+	7550 3300 8100 3300
 Wire Wire Line
-	7600 3450 8150 3450
+	7550 3400 8100 3400
 Wire Wire Line
-	7600 3550 8150 3550
-Text Label 7600 3150 0    50   ~ 0
+	7550 3500 8100 3500
+Text Label 7550 3100 0    50   ~ 0
 RXD2
-Text Label 7600 3250 0    50   ~ 0
+Text Label 7550 3200 0    50   ~ 0
 TXD1
-Text Label 7600 3350 0    50   ~ 0
+Text Label 7550 3300 0    50   ~ 0
 SleepRQ
-Text Label 7600 3450 0    50   ~ 0
+Text Label 7550 3400 0    50   ~ 0
 SLEEP
-Text Label 7600 3550 0    50   ~ 0
+Text Label 7550 3500 0    50   ~ 0
 CTS
 $Comp
 L power:+3.3V #PWR?
 U 1 1 5B7892DF
-P 4700 3150
-F 0 "#PWR?" H 4700 3000 50  0001 C CNN
-F 1 "+3.3V" H 4715 3323 50  0000 C CNN
-F 2 "" H 4700 3150 50  0001 C CNN
-F 3 "" H 4700 3150 50  0001 C CNN
-	1    4700 3150
+P 5000 3100
+F 0 "#PWR?" H 5000 2950 50  0001 C CNN
+F 1 "+3.3V" H 5015 3273 50  0000 C CNN
+F 2 "" H 5000 3100 50  0001 C CNN
+F 3 "" H 5000 3100 50  0001 C CNN
+	1    5000 3100
 	1    0    0    -1
 $EndComp
+Wire Wire Line
+	6750 3300 7100 3300
+Wire Wire Line
+	6750 3100 7100 3100
+Wire Wire Line
+	7550 3600 8100 3600
+Text HLabel 8100 3600 2    50   Output ~ 0
+RSSI
+Text Label 7550 3600 0    50   ~ 0
+RSSI
+Text Label 7100 3300 2    50   ~ 0
+RSSI
+Wire Wire Line
+	5350 3500 5000 3500
+Wire Wire Line
+	5000 3500 5000 3600
+$Comp
+L power:GND #PWR?
+U 1 1 5B7CBBC2
+P 5000 3600
+F 0 "#PWR?" H 5000 3350 50  0001 C CNN
+F 1 "GND" H 5005 3427 50  0000 C CNN
+F 2 "" H 5000 3600 50  0001 C CNN
+F 3 "" H 5000 3600 50  0001 C CNN
+	1    5000 3600
+	1    0    0    -1
+$EndComp
+Wire Wire Line
+	5000 3200 5350 3200
+Wire Wire Line
+	6750 3900 7100 3900
+Text Label 7100 3900 2    50   ~ 0
+RTS
+Text Label 7550 3700 0    50   ~ 0
+RTS
+Wire Wire Line
+	7550 3700 8100 3700
+Text HLabel 8100 3700 2    50   Input ~ 0
+RTS
 $EndSCHEMATC
