File: sch/proyecto.sch (KiCad schematic (older format))
At the start: 1 part

Commit message: cambios sch
Connections:
- wire segments 18 -> 21
Changed lines of the file:
@@
 $EndSheet
 $Sheet
-S 5550 1900 1800 3750
-U 5B71A3A9
-F0 "LPC" 50
-F1 "LPC.sch" 50
-F2 "TXD3" O R 7350 3800 50
-F3 "RXD3" I R 7350 4000 50
-F4 "SDA0" B R 7350 2750 50
-F5 "SCL0" B R 7350 3050 50
-F6 "RXD2" I R 7350 2050 50
-F7 "TXD2" O R 7350 2200 50
-F8 "MOSI1" O R 7350 4950 50
-F9 "MISO1" I R 7350 5100 50
-F10 "SCK1" O R 7350 5250 50
-F11 "SSEL1" O R 7350 5400 50
-F12 "DIR" I R 7350 4200 50
-$EndSheet
-$Sheet
-S 8100 1650 1550 750
+S 8100 1350 1500 1050
 U 5B71E2E3
 F0 "ZigBee" 50
 F1 "ZigBee.sch" 50
-F2 "TXD2" I L 8100 2200 50
-F3 "RXD2" O L 8100 2050 50
+F2 "TXD2" I L 8100 1650 50
+F3 "RXD2" O L 8100 1500 50
+F4 "SLRQ" I L 8100 2150 50
+F5 "SLEEP" O L 8100 2050 50
+F6 "CTS" O L 8100 1800 50
+F7 "RSSI" O L 8100 2250 50
+F8 "RTS" I L 8100 1950 50
 $EndSheet
 $Sheet
@@
 F3 "SCL0" B L 8100 3050 50
 $EndSheet
-Wire Wire Line
-	7350 2750 8100 2750
-Wire Wire Line
-	8100 3050 7350 3050
 $Sheet
 S 8100 3550 1550 900
@@
 F4 "DIR" O L 8100 4200 50
 $EndSheet
-Wire Wire Line
-	8100 3800 7350 3800
-Wire Wire Line
-	7350 4000 8100 4000
 $Sheet
 S 8100 4850 1500 850
@@
 $EndSheet
 Wire Wire Line
-	7350 4950 8100 4950
-Wire Wire Line
-	8100 5100 7350 5100
-Wire Wire Line
-	7350 5250 8100 5250
-Wire Wire Line
-	8100 5400 7350 5400
-Wire Wire Line
-	7350 2050 8100 2050
-Wire Wire Line
-	7350 2200 8100 2200
-Wire Wire Line
 	3600 4600 3900 4600
 $Sheet
@@
 $EndSheet
 Wire Wire Line
-	7350 4200 8100 4200
+	7400 1500 8100 1500
+Wire Wire Line
+	8100 1650 7400 1650
+Wire Wire Line
+	7400 2250 8100 2250
+Wire Wire Line
+	7400 3050 8100 3050
+Wire Wire Line
+	7400 2750 8100 2750
+Wire Wire Line
+	7400 3800 8100 3800
+Wire Wire Line
+	8100 4000 7400 4000
+Wire Wire Line
+	7400 4950 8100 4950
+Wire Wire Line
+	8100 5100 7400 5100
+Wire Wire Line
+	7400 5250 8100 5250
+Wire Wire Line
+	8100 5400 7400 5400
+$Sheet
+S 5550 1350 1850 4350
+U 5B71A3A9
+F0 "LPC" 50
+F1 "LPC.sch" 50
+F2 "TXD3" O R 7400 3800 50
+F3 "RXD3" I R 7400 4000 50
+F4 "SDA0" B R 7400 2750 50
+F5 "SCL0" B R 7400 3050 50
+F6 "MOSI1" O R 7400 4950 50
+F7 "MISO1" I R 7400 5100 50
+F8 "SCK1" O R 7400 5250 50
+F9 "SSEL1" O R 7400 5400 50
+F10 "DIR" I R 7400 4200 50
+F11 "CAP2.1" I R 7400 2250 50
+F12 "TXD1" O R 7400 1650 50
+F13 "RXD1" I R 7400 1500 50
+F14 "CTS1" I R 7400 1800 50
+F15 "RTS1" O R 7400 1950 50
+$EndSheet
+Wire Wire Line
+	7400 1800 8100 1800
+Wire Wire Line
+	8100 1950 7400 1950
+Wire Wire Line
+	7400 4200 8100 4200
 $EndSCHEMATC
