File: sch/regulador.sch (KiCad schematic (older format))
At the start: 6 parts

Commit message: cambios sch
Parts:
- removed C? (x2): 10uF, symbol Device:C
- removed U?: AIC1117-33PT, symbol aic1117:AIC1117-33PT
- added C? (x2): CP, symbol Device:CP
- added D?: D_Schottky, symbol Device:D_Schottky
- added L?: 330u, symbol Device:L
- added U?: LM2575-3.3, symbol lm2575:LM2575-3.3
Connections:
- wire segments 18 -> 27
