File: pcbs/cargador/regulador.sch (KiCad schematic (older format))
At the start: 8 parts, among them U2 LM2940-5V, U3 LM2575-3.3

Commit message: pdfs realizados
Other:
- note added: "3V3 & 5V"
- note added: "IMPORANTE:\nLos capacitores y diodos lo más cerca posible de los puertos en el pcb."
- note added: "REGULADORES DE VOLTAJE"
- moved on the sheet: C5, C6, C7, C8, D2, L1, U2, U3

Commit message: correcciones en los pdfs de los pcb
Parts:
- C8: footprint Capacitors_SMD:CP_Elec_10x10.5 -> Capacitors_SMD:CP_Elec_6.3x7.7
Changed lines of the file:
@@
 F 0 "C8" H 7275 3500 50  0000 L CNN
 F 1 "330u 50V" H 7275 3300 50  0000 L CNN
-F 2 "Capacitors_SMD:CP_Elec_10x10.5" H 7288 3250 50  0001 C CNN
+F 2 "Capacitors_SMD:CP_Elec_6.3x7.7" H 7288 3250 50  0001 C CNN
 F 3 "" H 7250 3400 50  0001 C CNN
 	1    7250 3400
