File: pcbs/pbase/Display.sch (KiCad schematic (older format))
At the start: 1 part

Commit message: update 11 sep
Parts:
- added R? (x2): 2k2, symbol R
Connections:
- net +5V: now also R?.1, R?.1
- net SCL2: now also R?.2
- net SDA2: now also R?.2
Other:
- note added: "# Se agregaron estos resistores de pull-up\n"
- note added: "# VALORES ARBITRARIOS"
Changed lines of the file:
@@
 Text Label 6250 4050 2    60   ~ 0
 GND
-Text HLabel 6800 3850 2    60   BiDi ~ 0
+Text HLabel 7750 3850 2    60   BiDi ~ 0
 SDA2
-Text HLabel 6800 3950 2    60   BiDi ~ 0
+Text HLabel 7750 3950 2    60   BiDi ~ 0
 SCL2
 $Comp
 L +5V #PWR?
 U 1 1 5B964359
-P 6800 3550
-F 0 "#PWR?" H 6800 3400 50  0001 C CNN
-F 1 "+5V" H 6800 3690 50  0000 C CNN
-F 2 "" H 6800 3550 50  0001 C CNN
-F 3 "" H 6800 3550 50  0001 C CNN
-	1    6800 3550
+P 6800 3350
+F 0 "#PWR?" H 6800 3200 50  0001 C CNN
+F 1 "+5V" H 6800 3490 50  0000 C CNN
+F 2 "" H 6800 3350 50  0001 C CNN
+F 3 "" H 6800 3350 50  0001 C CNN
+	1    6800 3350
 	1    0    0    -1
 $EndComp
@@
 	4850 3950 5250 3950
 Wire Wire Line
-	6250 3850 6800 3850
+	6250 3850 7150 3850
 Wire Wire Line
-	6250 3950 6800 3950
+	7150 3850 7750 3850
+Wire Wire Line
+	6250 3950 7550 3950
+Wire Wire Line
+	7550 3950 7750 3950
 Wire Wire Line
 	6250 3750 6800 3750
@@
 	6800 4050 6800 4250
 Wire Wire Line
-	6800 3750 6800 3550
+	6800 3750 6800 3350
 Text Notes 5700 2800 0    60   ~ 12
 Display
+$Comp
+L R R?
+U 1 1 5B97E047
+P 7150 3550
+F 0 "R?" H 7300 3600 50  0000 C CNN
+F 1 "2k2" H 7300 3500 50  0000 C CNN
+F 2 "" V 7080 3550 50  0001 C CNN
+F 3 "" H 7150 3550 50  0001 C CNN
+	1    7150 3550
+	1    0    0    -1
+$EndComp
+$Comp
+L R R?
+U 1 1 5B97E06A
+P 7550 3550
+F 0 "R?" H 7700 3600 50  0000 C CNN
+F 1 "2k2" H 7700 3500 50  0000 C CNN
+F 2 "" V 7480 3550 50  0001 C CNN
+F 3 "" H 7550 3550 50  0001 C CNN
+	1    7550 3550
+	1    0    0    -1
+$EndComp
+Wire Wire Line
+	7150 3700 7150 3850
+Connection ~ 7150 3850
+Wire Wire Line
+	7550 3700 7550 3950
+Connection ~ 7550 3950
+Text Notes 7800 3550 0    60   ~ 0
+# Se agregaron estos resistores de pull-up\n
+$Comp
+L +5V #PWR?
+U 1 1 5B97FB09
+P 7150 3350
+F 0 "#PWR?" H 7150 3200 50  0001 C CNN
+F 1 "+5V" H 7150 3490 50  0000 C CNN
+F 2 "" H 7150 3350 50  0001 C CNN
+F 3 "" H 7150 3350 50  0001 C CNN
+	1    7150 3350
+	1    0    0    -1
+$EndComp
+$Comp
+L +5V #PWR?
+U 1 1 5B97FB23
+P 7550 3350
+F 0 "#PWR?" H 7550 3200 50  0001 C CNN
+F 1 "+5V" H 7550 3490 50  0000 C CNN
+F 2 "" H 7550 3350 50  0001 C CNN
+F 3 "" H 7550 3350 50  0001 C CNN
+	1    7550 3350
+	1    0    0    -1
+$EndComp
+Wire Wire Line
+	7150 3350 7150 3400
+Wire Wire Line
+	7550 3350 7550 3400
+Text Notes 8200 3650 0    60   ~ 0
+# VALORES ARBITRARIOS
 $EndSCHEMATC

Commit message: Test points
Parts:
- R?: value 2k2 -> RD1
- R?: value 2k2 -> RD2
Other:
- note removed: "# Se agregaron estos resistores de pull-up\n"
- note removed: "# VALORES ARBITRARIOS"
Changed lines of the file:
@@
 	4850 3950 5250 3950
 Wire Wire Line
-	6250 3850 7150 3850
+	6250 3850 7750 3850
 Wire Wire Line
-	7150 3850 7750 3850
-Wire Wire Line
-	6250 3950 7550 3950
-Wire Wire Line
-	7550 3950 7750 3950
+	6250 3950 7750 3950
 Wire Wire Line
 	6250 3750 6800 3750
@@
 P 7150 3550
 F 0 "R?" H 7300 3600 50  0000 C CNN
-F 1 "2k2" H 7300 3500 50  0000 C CNN
+F 1 "RD1" H 7300 3500 50  0000 C CNN
 F 2 "" V 7080 3550 50  0001 C CNN
 F 3 "" H 7150 3550 50  0001 C CNN
@@
 P 7550 3550
 F 0 "R?" H 7700 3600 50  0000 C CNN
-F 1 "2k2" H 7700 3500 50  0000 C CNN
+F 1 "RD2" H 7700 3500 50  0000 C CNN
 F 2 "" V 7480 3550 50  0001 C CNN
 F 3 "" H 7550 3550 50  0001 C CNN
@@
 	7550 3700 7550 3950
 Connection ~ 7550 3950
-Text Notes 7800 3550 0    60   ~ 0
-# Se agregaron estos resistores de pull-up\n
 $Comp
 L +5V #PWR?
@@
 Wire Wire Line
 	7550 3350 7550 3400
-Text Notes 8200 3650 0    60   ~ 0
-# VALORES ARBITRARIOS
 $EndSCHEMATC

Commit message: sch annotate v1.1
Parts:
- gave numbers to parts that had none: 3
Changed lines of the file:
@@
 Comment1 ""
 Comment2 ""
-Comment3 ""
-Comment4 ""
+Comment3 "Si alguno de los dos dispositivos ya los incorpora, quitarlos."
+Comment4 "RD1 y RD2 deben calcularse para realizar la comunicación I2C."
 $EndDescr
 $Comp
-L Conn_01x04 J?
+L Conn_01x04 J2
 U 1 1 5B962FE7
 P 5450 3850
-F 0 "J?" H 5450 4050 50  0000 C CNN
+F 0 "J2" H 5450 4050 50  0000 C CNN
 F 1 "Conn_01x04" H 5450 3550 50  0000 C CNN
 F 2 "" H 5450 3850 50  0001 C CNN
@@
 SCL2
 $Comp
-L +5V #PWR018
+L +5V #PWR18
 U 1 1 5B964359
 P 6800 3350
-F 0 "#PWR018" H 6800 3200 50  0001 C CNN
+F 0 "#PWR18" H 6800 3200 50  0001 C CNN
 F 1 "+5V" H 6800 3490 50  0000 C CNN
 F 2 "" H 6800 3350 50  0001 C CNN
@@
 $EndComp
 $Comp
-L GND #PWR019
+L GND #PWR19
 U 1 1 5B96436F
 P 6800 4250
-F 0 "#PWR019" H 6800 4000 50  0001 C CNN
+F 0 "#PWR19" H 6800 4000 50  0001 C CNN
 F 1 "GND" H 6800 4100 50  0000 C CNN
 F 2 "" H 6800 4250 50  0001 C CNN
@@
 Display
 $Comp
-L R R?
+L R R6
 U 1 1 5B97E047
 P 7150 3550
-F 0 "R?" H 7300 3600 50  0000 C CNN
+F 0 "R6" H 7300 3600 50  0000 C CNN
 F 1 "RD1" H 7300 3500 50  0000 C CNN
 F 2 "" V 7080 3550 50  0001 C CNN
@@
 $EndComp
 $Comp
-L R R?
+L R R7
 U 1 1 5B97E06A
 P 7550 3550
-F 0 "R?" H 7700 3600 50  0000 C CNN
+F 0 "R7" H 7700 3600 50  0000 C CNN
 F 1 "RD2" H 7700 3500 50  0000 C CNN
 F 2 "" V 7480 3550 50  0001 C CNN
@@
 Connection ~ 7550 3950
 $Comp
-L +5V #PWR020
+L +5V #PWR20
 U 1 1 5B97FB09
 P 7150 3350
-F 0 "#PWR020" H 7150 3200 50  0001 C CNN
+F 0 "#PWR20" H 7150 3200 50  0001 C CNN
 F 1 "+5V" H 7150 3490 50  0000 C CNN
 F 2 "" H 7150 3350 50  0001 C CNN
@@
 $EndComp
 $Comp
-L +5V #PWR021
+L +5V #PWR21
 U 1 1 5B97FB23
 P 7550 3350
-F 0 "#PWR021" H 7550 3200 50  0001 C CNN
+F 0 "#PWR21" H 7550 3200 50  0001 C CNN
 F 1 "+5V" H 7550 3490 50  0000 C CNN
 F 2 "" H 7550 3350 50  0001 C CNN

Commit message: pbase pcb inicio
Parts:
- J2: footprint (none) -> Socket_Strips:Socket_Strip_Straight_1x04_Pitch2.54mm
- R6, R7: footprint (none) -> Resistors_SMD:R_0805_HandSoldering
Changed lines of the file:
@@
 F 0 "J2" H 5450 4050 50  0000 C CNN
 F 1 "Conn_01x04" H 5450 3550 50  0000 C CNN
-F 2 "" H 5450 3850 50  0001 C CNN
+F 2 "Socket_Strips:Socket_Strip_Straight_1x04_Pitch2.54mm" H 5450 3850 50  0001 C CNN
 F 3 "" H 5450 3850 50  0001 C CNN
 	1    5450 3850
@@
 SCL2
 $Comp
-L +5V #PWR18
+L +5V #PWR018
 U 1 1 5B964359
 P 6800 3350
-F 0 "#PWR18" H 6800 3200 50  0001 C CNN
+F 0 "#PWR018" H 6800 3200 50  0001 C CNN
 F 1 "+5V" H 6800 3490 50  0000 C CNN
 F 2 "" H 6800 3350 50  0001 C CNN
@@
 $EndComp
 $Comp
-L GND #PWR19
+L GND #PWR019
 U 1 1 5B96436F
 P 6800 4250
-F 0 "#PWR19" H 6800 4000 50  0001 C CNN
+F 0 "#PWR019" H 6800 4000 50  0001 C CNN
 F 1 "GND" H 6800 4100 50  0000 C CNN
 F 2 "" H 6800 4250 50  0001 C CNN
@@
 F 0 "R6" H 7300 3600 50  0000 C CNN
 F 1 "RD1" H 7300 3500 50  0000 C CNN
-F 2 "" V 7080 3550 50  0001 C CNN
+F 2 "Resistors_SMD:R_0805_HandSoldering" V 7080 3550 50  0001 C CNN
 F 3 "" H 7150 3550 50  0001 C CNN
 	1    7150 3550
@@
 F 0 "R7" H 7700 3600 50  0000 C CNN
 F 1 "RD2" H 7700 3500 50  0000 C CNN
-F 2 "" V 7480 3550 50  0001 C CNN
+F 2 "Resistors_SMD:R_0805_HandSoldering" V 7480 3550 50  0001 C CNN
 F 3 "" H 7550 3550 50  0001 C CNN
 	1    7550 3550
@@
 Connection ~ 7550 3950
 $Comp
-L +5V #PWR20
+L +5V #PWR020
 U 1 1 5B97FB09
 P 7150 3350
-F 0 "#PWR20" H 7150 3200 50  0001 C CNN
+F 0 "#PWR020" H 7150 3200 50  0001 C CNN
 F 1 "+5V" H 7150 3490 50  0000 C CNN
 F 2 "" H 7150 3350 50  0001 C CNN
@@
 $EndComp
 $Comp
-L +5V #PWR21
+L +5V #PWR021
 U 1 1 5B97FB23
 P 7550 3350
-F 0 "#PWR21" H 7550 3200 50  0001 C CNN
+F 0 "#PWR021" H 7550 3200 50  0001 C CNN
 F 1 "+5V" H 7550 3490 50  0000 C CNN
 F 2 "" H 7550 3350 50  0001 C CNN

Commit message: pdfs realizados
Other:
- note added: "IMPORTANTE.\nRD1 y RD2 deben calcularse para realizar la comunicación I2C.\nSi alguno de los dos dispositivos ya los incorpora, quitarlos."
Changed lines of the file:
@@
 encoding utf-8
 Sheet 7 8
-Title "Display"
-Date "2018-09-10"
+Title "Diagrama de bloques "
+Date "2018-10-30"
 Rev "A"
 Comp "UTN - FRBA"
-Comment1 ""
+Comment1 "Autores: Alegre M. E., Bautista L., Tarazona L."
 Comment2 ""
-Comment3 "Si alguno de los dos dispositivos ya los incorpora, quitarlos."
-Comment4 "RD1 y RD2 deben calcularse para realizar la comunicación I2C."
+Comment3 ""
+Comment4 "Display OLED I2C"
 $EndDescr
 $Comp
@@
 	1    0    0    -1
 $EndComp
-Text Notes 4700 3100 0    60   ~ 0
+Text Notes 4750 2300 0    60   ~ 0
 Display Oled 0.96 Azul 128x64 I2c Ssd1306 Nubbeo
 Text Label 4850 4050 2    60   ~ 0
@@
 	1    0    0    -1
 $EndComp
-Wire Wire Line
-	4850 3750 5250 3750
-Wire Wire Line
-	4850 4050 5250 4050
-Wire Wire Line
-	4850 3850 5250 3850
-Wire Wire Line
-	4850 3950 5250 3950
-Wire Wire Line
-	6250 3850 7750 3850
-Wire Wire Line
-	6250 3950 7750 3950
-Wire Wire Line
-	6250 3750 6800 3750
-Wire Wire Line
-	6250 4050 6800 4050
-Wire Wire Line
-	6800 4050 6800 4250
-Wire Wire Line
-	6800 3750 6800 3350
-Text Notes 5700 2800 0    60   ~ 12
+Text Notes 5500 1950 0    157  ~ 31
 Display
 $Comp
@@
 	1    0    0    -1
 $EndComp
-Wire Wire Line
-	7150 3700 7150 3850
-Connection ~ 7150 3850
-Wire Wire Line
-	7550 3700 7550 3950
-Connection ~ 7550 3950
 $Comp
 L +5V #PWR020
@@
 	1    0    0    -1
 $EndComp
+Text Notes 1150 6900 0    60   ~ 12
+IMPORTANTE.\nRD1 y RD2 deben calcularse para realizar la comunicación I2C.\nSi alguno de los dos dispositivos ya los incorpora, quitarlos.
+Wire Wire Line
+	4850 3750 5250 3750
+Wire Wire Line
+	4850 4050 5250 4050
+Wire Wire Line
+	4850 3850 5250 3850
+Wire Wire Line
+	4850 3950 5250 3950
+Wire Wire Line
+	6250 3850 7750 3850
+Wire Wire Line
+	6250 3950 7750 3950
+Wire Wire Line
+	6250 3750 6800 3750
+Wire Wire Line
+	6250 4050 6800 4050
+Wire Wire Line
+	6800 4050 6800 4250
+Wire Wire Line
+	6800 3750 6800 3350
+Wire Wire Line
+	7150 3700 7150 3850
+Connection ~ 7150 3850
+Wire Wire Line
+	7550 3700 7550 3950
+Connection ~ 7550 3950
 Wire Wire Line
 	7150 3350 7150 3400
 Wire Wire Line
 	7550 3350 7550 3400
+Wire Notes Line
+	1100 6550 1100 7000
+Wire Notes Line
+	1100 7000 4200 7000
+Wire Notes Line
+	4200 7000 4200 6550
+Wire Notes Line
+	4200 6550 1100 6550
 $EndSCHEMATC
