File: pcbs/pbase/TarjetaSD.sch (KiCad schematic (older format))
At the start: 7 parts

Commit message: sch annotate v1.1
Parts:
- gave numbers to parts that had none: 7
Changed lines of the file:
@@
 $EndDescr
 $Comp
-L SD_Card J?
+L SD_Card J1
 U 1 1 5B95F793
 P 5650 3000
-F 0 "J?" H 5000 3550 50  0000 C CNN
+F 0 "J1" H 5000 3550 50  0000 C CNN
 F 1 "SD_Card" H 6250 2450 50  0000 C CNN
 F 2 "10067847-001" H 5850 3350 50  0001 C CNN
@@
 $EndComp
 $Comp
-L +3V3 #PWR013
+L +3V3 #PWR13
 U 1 1 5B95F880
 P 3950 2150
-F 0 "#PWR013" H 3950 2000 50  0001 C CNN
+F 0 "#PWR13" H 3950 2000 50  0001 C CNN
 F 1 "+3V3" H 3950 2290 50  0000 C CNN
 F 2 "" H 3950 2150 50  0001 C CNN
@@
 $EndComp
 $Comp
-L GND #PWR014
+L GND #PWR14
 U 1 1 5B95F899
 P 3950 3850
-F 0 "#PWR014" H 3950 3600 50  0001 C CNN
+F 0 "#PWR14" H 3950 3600 50  0001 C CNN
 F 1 "GND" H 3950 3700 50  0000 C CNN
 F 2 "" H 3950 3850 50  0001 C CNN
@@
 $EndComp
 $Comp
-L CP C?
+L CP C1
 U 1 1 5B95F982
 P 7450 2750
-F 0 "C?" H 7475 2850 50  0000 L CNN
+F 0 "C1" H 7475 2850 50  0000 L CNN
 F 1 "1uF x 16V" H 7475 2650 50  0000 L CNN
 F 2 "" H 7488 2600 50  0001 C CNN
@@
 $EndComp
 $Comp
-L C C?
+L C C2
 U 1 1 5B95F99B
 P 8050 2750
-F 0 "C?" H 8075 2850 50  0000 L CNN
+F 0 "C2" H 8075 2850 50  0000 L CNN
 F 1 "100n" H 8075 2650 50  0000 L CNN
 F 2 "" H 8088 2600 50  0001 C CNN
@@
 $EndComp
 $Comp
-L +3V3 #PWR015
+L +3V3 #PWR16
 U 1 1 5B95FAF6
 P 7450 2200
-F 0 "#PWR015" H 7450 2050 50  0001 C CNN
+F 0 "#PWR16" H 7450 2050 50  0001 C CNN
 F 1 "+3V3" H 7450 2340 50  0000 C CNN
 F 2 "" H 7450 2200 50  0001 C CNN
@@
 $EndComp
 $Comp
-L GND #PWR016
+L GND #PWR17
 U 1 1 5B95FC27
 P 7450 3400
-F 0 "#PWR016" H 7450 3150 50  0001 C CNN
+F 0 "#PWR17" H 7450 3150 50  0001 C CNN
 F 1 "GND" H 7450 3250 50  0000 C CNN
 F 2 "" H 7450 3400 50  0001 C CNN
@@
 data1
 $Comp
-L R R?
+L R R2
 U 1 1 5B96095B
 P 4950 4500
-F 0 "R?" H 5100 4550 50  0000 C CNN
+F 0 "R2" H 5100 4550 50  0000 C CNN
 F 1 "10K" H 5100 4450 50  0000 C CNN
 F 2 "" V 4880 4500 50  0001 C CNN
@@
 $EndComp
 $Comp
-L R R?
+L R R3
 U 1 1 5B96098C
 P 5350 4500
-F 0 "R?" H 5500 4550 50  0000 C CNN
+F 0 "R3" H 5500 4550 50  0000 C CNN
 F 1 "10K" H 5500 4450 50  0000 C CNN
 F 2 "" V 5280 4500 50  0001 C CNN
@@
 $EndComp
 $Comp
-L R R?
+L R R4
 U 1 1 5B9609B5
 P 5750 4500
-F 0 "R?" H 5900 4550 50  0000 C CNN
+F 0 "R4" H 5900 4550 50  0000 C CNN
 F 1 "33K" H 5900 4450 50  0000 C CNN
 F 2 "" V 5680 4500 50  0001 C CNN
@@
 $EndComp
 $Comp
-L R R?
+L R R5
 U 1 1 5B9609E0
 P 6150 4500
-F 0 "R?" H 6300 4550 50  0000 C CNN
+F 0 "R5" H 6300 4550 50  0000 C CNN
 F 1 "33K" H 6300 4450 50  0000 C CNN
 F 2 "" V 6080 4500 50  0001 C CNN
@@
 $EndComp
 $Comp
-L +3V3 #PWR017
+L +3V3 #PWR15
 U 1 1 5B960A05
 P 6250 4150
-F 0 "#PWR017" H 6250 4000 50  0001 C CNN
+F 0 "#PWR15" H 6250 4000 50  0001 C CNN
 F 1 "+3V3" H 6250 4290 50  0000 C CNN
 F 2 "" H 6250 4150 50  0001 C CNN

Commit message: pbase pcb inicio
Parts:
- C1: footprint (none) -> Capacitors_Tantalum_SMD:CP_Tantalum_Case-A_EIA-3216-18_Hand
- C2: footprint (none) -> Capacitors_SMD:C_0805_HandSoldering
- J1: footprint 10067847-001 -> Connectors:SD_Card_Receptacle
- R2, R3, R4, R5: footprint (none) -> Resistors_SMD:R_0805_HandSoldering
Changed lines of the file:
@@
 F 0 "J1" H 5000 3550 50  0000 C CNN
 F 1 "SD_Card" H 6250 2450 50  0000 C CNN
-F 2 "10067847-001" H 5850 3350 50  0001 C CNN
+F 2 "Connectors:SD_Card_Receptacle" H 5850 3350 50  0001 C CNN
 F 3 "" H 5650 3000 50  0001 C CNN
 	1    5650 3000
@@
 $EndComp
 $Comp
-L +3V3 #PWR13
+L +3V3 #PWR013
 U 1 1 5B95F880
 P 3950 2150
-F 0 "#PWR13" H 3950 2000 50  0001 C CNN
+F 0 "#PWR013" H 3950 2000 50  0001 C CNN
 F 1 "+3V3" H 3950 2290 50  0000 C CNN
 F 2 "" H 3950 2150 50  0001 C CNN
@@
 $EndComp
 $Comp
-L GND #PWR14
+L GND #PWR014
 U 1 1 5B95F899
 P 3950 3850
-F 0 "#PWR14" H 3950 3600 50  0001 C CNN
+F 0 "#PWR014" H 3950 3600 50  0001 C CNN
 F 1 "GND" H 3950 3700 50  0000 C CNN
 F 2 "" H 3950 3850 50  0001 C CNN
@@
 F 0 "C1" H 7475 2850 50  0000 L CNN
 F 1 "1uF x 16V" H 7475 2650 50  0000 L CNN
-F 2 "" H 7488 2600 50  0001 C CNN
+F 2 "Capacitors_Tantalum_SMD:CP_Tantalum_Case-A_EIA-3216-18_Hand" H 7488 2600 50  0001 C CNN
 F 3 "" H 7450 2750 50  0001 C CNN
 	1    7450 2750
@@
 F 0 "C2" H 8075 2850 50  0000 L CNN
 F 1 "100n" H 8075 2650 50  0000 L CNN
-F 2 "" H 8088 2600 50  0001 C CNN
+F 2 "Capacitors_SMD:C_0805_HandSoldering" H 8088 2600 50  0001 C CNN
 F 3 "" H 8050 2750 50  0001 C CNN
 	1    8050 2750
@@
 $EndComp
 $Comp
-L +3V3 #PWR16
+L +3V3 #PWR015
 U 1 1 5B95FAF6
 P 7450 2200
-F 0 "#PWR16" H 7450 2050 50  0001 C CNN
+F 0 "#PWR015" H 7450 2050 50  0001 C CNN
 F 1 "+3V3" H 7450 2340 50  0000 C CNN
 F 2 "" H 7450 2200 50  0001 C CNN
@@
 $EndComp
 $Comp
-L GND #PWR17
+L GND #PWR016
 U 1 1 5B95FC27
 P 7450 3400
-F 0 "#PWR17" H 7450 3150 50  0001 C CNN
+F 0 "#PWR016" H 7450 3150 50  0001 C CNN
 F 1 "GND" H 7450 3250 50  0000 C CNN
 F 2 "" H 7450 3400 50  0001 C CNN
@@
 F 0 "R2" H 5100 4550 50  0000 C CNN
 F 1 "10K" H 5100 4450 50  0000 C CNN
-F 2 "" V 4880 4500 50  0001 C CNN
+F 2 "Resistors_SMD:R_0805_HandSoldering" V 4880 4500 50  0001 C CNN
 F 3 "" H 4950 4500 50  0001 C CNN
 	1    4950 4500
@@
 F 0 "R3" H 5500 4550 50  0000 C CNN
 F 1 "10K" H 5500 4450 50  0000 C CNN
-F 2 "" V 5280 4500 50  0001 C CNN
+F 2 "Resistors_SMD:R_0805_HandSoldering" V 5280 4500 50  0001 C CNN
 F 3 "" H 5350 4500 50  0001 C CNN
 	1    5350 4500
@@
 F 0 "R4" H 5900 4550 50  0000 C CNN
 F 1 "33K" H 5900 4450 50  0000 C CNN
-F 2 "" V 5680 4500 50  0001 C CNN
+F 2 "Resistors_SMD:R_0805_HandSoldering" V 5680 4500 50  0001 C CNN
 F 3 "" H 5750 4500 50  0001 C CNN
 	1    5750 4500
@@
 F 0 "R5" H 6300 4550 50  0000 C CNN
 F 1 "33K" H 6300 4450 50  0000 C CNN
-F 2 "" V 6080 4500 50  0001 C CNN
+F 2 "Resistors_SMD:R_0805_HandSoldering" V 6080 4500 50  0001 C CNN
 F 3 "" H 6150 4500 50  0001 C CNN
 	1    6150 4500
@@
 $EndComp
 $Comp
-L +3V3 #PWR15
+L +3V3 #PWR017
 U 1 1 5B960A05
 P 6250 4150
-F 0 "#PWR15" H 6250 4000 50  0001 C CNN
+F 0 "#PWR017" H 6250 4000 50  0001 C CNN
 F 1 "+3V3" H 6250 4290 50  0000 C CNN
 F 2 "" H 6250 4150 50  0001 C CNN

Commit message: PCB PLACING V1
Parts:
- J1: footprint Connectors:SD_Card_Receptacle -> footprints:SD_TE_2041021
Changed lines of the file:
@@
 F 0 "J1" H 5000 3550 50  0000 C CNN
 F 1 "SD_Card" H 6250 2450 50  0000 C CNN
-F 2 "Connectors:SD_Card_Receptacle" H 5850 3350 50  0001 C CNN
+F 2 "footprints:SD_TE_2041021" H 5850 3350 50  0001 C CNN
 F 3 "" H 5650 3000 50  0001 C CNN
 	1    5650 3000

Commit message: pcb fin 1
Parts:
- J1: footprint footprints:SD_TE_2041021 -> footprints:SD_TE_2041021_edit
Changed lines of the file:
@@
 F 0 "J1" H 5000 3550 50  0000 C CNN
 F 1 "SD_Card" H 6250 2450 50  0000 C CNN
-F 2 "footprints:SD_TE_2041021" H 5850 3350 50  0001 C CNN
+F 2 "footprints:SD_TE_2041021_edit" H 5850 3350 50  0001 C CNN
 F 3 "" H 5650 3000 50  0001 C CNN
 	1    5650 3000

Commit message: pdfs realizados
Changed lines of the file:
@@
 encoding utf-8
 Sheet 6 8
-Title "Tarjeta SD"
-Date "2018-09-10"
+Title "Diagrama de bloques "
+Date "2018-10-30"
 Rev "A"
 Comp "UTN - FRBA"
-Comment1 ""
+Comment1 "Autores: Alegre M. E., Bautista L., Tarazona L."
 Comment2 ""
 Comment3 ""
-Comment4 ""
+Comment4 "Tarjeta SD"
 $EndDescr
 $Comp
@@
 Text HLabel 6250 5200 2    60   Input ~ 0
 SCK1
-Text Notes 5550 2000 0    60   ~ 12
+Text Notes 5250 1550 0    157  ~ 31
 Tarjeta SD\n
 $EndSCHEMATC
