File: pcbs/pbase/pwr.sch (KiCad schematic (older format))
At the start: 1 part

Commit message: update 11 sep
Parts:
- added TP? (x2): TEST, symbol TEST
Connections:
- net +3V3: now also TP?.1
- net +5V: now also TP?.1
Changed lines of the file:
@@
 L GND #PWR?
 U 1 1 5B96559F
-P 5600 4300
-F 0 "#PWR?" H 5600 4050 50  0001 C CNN
-F 1 "GND" H 5600 4150 50  0000 C CNN
-F 2 "" H 5600 4300 50  0001 C CNN
-F 3 "" H 5600 4300 50  0001 C CNN
-	1    5600 4300
+P 5600 4600
+F 0 "#PWR?" H 5600 4350 50  0001 C CNN
+F 1 "GND" H 5600 4450 50  0000 C CNN
+F 2 "" H 5600 4600 50  0001 C CNN
+F 3 "" H 5600 4600 50  0001 C CNN
+	1    5600 4600
 	1    0    0    -1
 $EndComp
@@
 L +3V3 #PWR?
 U 1 1 5B9655CB
-P 6450 3450
-F 0 "#PWR?" H 6450 3300 50  0001 C CNN
-F 1 "+3V3" H 6450 3590 50  0000 C CNN
-F 2 "" H 6450 3450 50  0001 C CNN
-F 3 "" H 6450 3450 50  0001 C CNN
-	1    6450 3450
+P 6850 3450
+F 0 "#PWR?" H 6850 3300 50  0001 C CNN
+F 1 "+3V3" H 6850 3590 50  0000 C CNN
+F 2 "" H 6850 3450 50  0001 C CNN
+F 3 "" H 6850 3450 50  0001 C CNN
+	1    6850 3450
 	1    0    0    -1
 $EndComp
@@
 L PWR_FLAG #FLG?
 U 1 1 5B965604
-P 6800 3850
-F 0 "#FLG?" H 6800 3925 50  0001 C CNN
-F 1 "PWR_FLAG" H 6800 4000 50  0000 C CNN
-F 2 "" H 6800 3850 50  0001 C CNN
-F 3 "" H 6800 3850 50  0001 C CNN
-	1    6800 3850
+P 7200 3850
+F 0 "#FLG?" H 7200 3925 50  0001 C CNN
+F 1 "PWR_FLAG" H 7200 4000 50  0000 C CNN
+F 2 "" H 7200 3850 50  0001 C CNN
+F 3 "" H 7200 3850 50  0001 C CNN
+	1    7200 3850
 	1    0    0    -1
 $EndComp
@@
 L PWR_FLAG #FLG?
 U 1 1 5B96561A
-P 6050 4200
-F 0 "#FLG?" H 6050 4275 50  0001 C CNN
-F 1 "PWR_FLAG" H 6050 4350 50  0000 C CNN
-F 2 "" H 6050 4200 50  0001 C CNN
-F 3 "" H 6050 4200 50  0001 C CNN
-	1    6050 4200
+P 6050 4300
+F 0 "#FLG?" H 6050 4375 50  0001 C CNN
+F 1 "PWR_FLAG" H 6050 4450 50  0000 C CNN
+F 2 "" H 6050 4300 50  0001 C CNN
+F 3 "" H 6050 4300 50  0001 C CNN
+	1    6050 4300
 	1    0    0    -1
 $EndComp
 Wire Wire Line
-	6450 3450 6450 4000
+	6850 3450 6850 4000
 Wire Wire Line
 	5800 3800 5800 3450
@@
 	6050 3800 6050 3650
 Wire Wire Line
-	6800 4000 6800 3850
+	7200 4000 7200 3850
 Wire Wire Line
-	6050 4250 6050 4200
+	6050 4500 6050 4300
 Wire Wire Line
 	5350 3700 5600 3700
 Wire Wire Line
-	5600 3700 5600 4300
+	5600 3700 5600 4600
 Wire Wire Line
 	5350 3900 5600 3900
 Connection ~ 5600 3900
+Connection ~ 5600 4500
 Wire Wire Line
-	6050 4250 5600 4250
-Connection ~ 5600 4250
-Wire Wire Line
-	5350 3800 6050 3800
+	5350 3800 6350 3800
 Connection ~ 5800 3800
 Wire Wire Line
-	5350 4000 6800 4000
-Connection ~ 6450 4000
+	5350 4000 7500 4000
+Connection ~ 6850 4000
+$Comp
+L TEST TP?
+U 1 1 5B982DEF
+P 6350 3750
+F 0 "TP?" H 6350 4050 50  0000 C BNN
+F 1 "TEST" H 6350 4000 50  0000 C CNN
+F 2 "" H 6350 3750 50  0001 C CNN
+F 3 "" H 6350 3750 50  0001 C CNN
+	1    6350 3750
+	1    0    0    -1
+$EndComp
+$Comp
+L TEST TP?
+U 1 1 5B982E1A
+P 7500 3950
+F 0 "TP?" H 7500 4250 50  0000 C BNN
+F 1 "TEST" H 7500 4200 50  0000 C CNN
+F 2 "" H 7500 3950 50  0001 C CNN
+F 3 "" H 7500 3950 50  0001 C CNN
+	1    7500 3950
+	1    0    0    -1
+$EndComp
+Wire Wire Line
+	7500 4000 7500 3950
+Connection ~ 7200 4000
+Wire Wire Line
+	6350 3800 6350 3750
+Connection ~ 6050 3800
+Wire Wire Line
+	6050 4500 5600 4500
 $EndSCHEMATC

Commit message: sch annotate v1.1
Parts:
- gave numbers to parts that had none: 3
Changed lines of the file:
@@
 Alimentación\n
 $Comp
-L Conn_01x04 J?
+L Conn_01x04 J3
 U 1 1 5B96555C
 P 5150 3900
-F 0 "J?" H 5150 4100 50  0000 C CNN
+F 0 "J3" H 5150 4100 50  0000 C CNN
 F 1 "Conn_01x04" H 5150 3600 50  0000 C CNN
 F 2 "" H 5150 3900 50  0001 C CNN
@@
 $EndComp
 $Comp
-L GND #PWR022
+L GND #PWR22
 U 1 1 5B96559F
 P 5600 4600
-F 0 "#PWR022" H 5600 4350 50  0001 C CNN
+F 0 "#PWR22" H 5600 4350 50  0001 C CNN
 F 1 "GND" H 5600 4450 50  0000 C CNN
 F 2 "" H 5600 4600 50  0001 C CNN
@@
 $EndComp
 $Comp
-L +5V #PWR023
+L +5V #PWR23
 U 1 1 5B9655B5
 P 5800 3450
-F 0 "#PWR023" H 5800 3300 50  0001 C CNN
+F 0 "#PWR23" H 5800 3300 50  0001 C CNN
 F 1 "+5V" H 5800 3590 50  0000 C CNN
 F 2 "" H 5800 3450 50  0001 C CNN
@@
 $EndComp
 $Comp
-L +3V3 #PWR024
+L +3V3 #PWR24
 U 1 1 5B9655CB
 P 6850 3450
-F 0 "#PWR024" H 6850 3300 50  0001 C CNN
+F 0 "#PWR24" H 6850 3300 50  0001 C CNN
 F 1 "+3V3" H 6850 3590 50  0000 C CNN
 F 2 "" H 6850 3450 50  0001 C CNN
@@
 $EndComp
 $Comp
-L PWR_FLAG #FLG025
+L PWR_FLAG #FLG1
 U 1 1 5B9655E1
 P 6050 3650
-F 0 "#FLG025" H 6050 3725 50  0001 C CNN
+F 0 "#FLG1" H 6050 3725 50  0001 C CNN
 F 1 "PWR_FLAG" H 6050 3800 50  0000 C CNN
 F 2 "" H 6050 3650 50  0001 C CNN
@@
 $EndComp
 $Comp
-L PWR_FLAG #FLG026
+L PWR_FLAG #FLG3
 U 1 1 5B965604
 P 7200 3850
-F 0 "#FLG026" H 7200 3925 50  0001 C CNN
+F 0 "#FLG3" H 7200 3925 50  0001 C CNN
 F 1 "PWR_FLAG" H 7200 4000 50  0000 C CNN
 F 2 "" H 7200 3850 50  0001 C CNN
@@
 $EndComp
 $Comp
-L PWR_FLAG #FLG027
+L PWR_FLAG #FLG2
 U 1 1 5B96561A
 P 6050 4300
-F 0 "#FLG027" H 6050 4375 50  0001 C CNN
+F 0 "#FLG2" H 6050 4375 50  0001 C CNN
 F 1 "PWR_FLAG" H 6050 4450 50  0000 C CNN
 F 2 "" H 6050 4300 50  0001 C CNN
@@
 Connection ~ 6850 4000
 $Comp
-L TEST TP?
+L TEST TP21
 U 1 1 5B982DEF
 P 6350 3750
-F 0 "TP?" H 6350 4050 50  0000 C BNN
+F 0 "TP21" H 6350 4050 50  0000 C BNN
 F 1 "TEST" H 6350 4000 50  0000 C CNN
 F 2 "" H 6350 3750 50  0001 C CNN
@@
 $EndComp
 $Comp
-L TEST TP?
+L TEST TP22
 U 1 1 5B982E1A
 P 7500 3950
-F 0 "TP?" H 7500 4250 50  0000 C BNN
+F 0 "TP22" H 7500 4250 50  0000 C BNN
 F 1 "TEST" H 7500 4200 50  0000 C CNN
 F 2 "" H 7500 3950 50  0001 C CNN

Commit message: pbase pcb inicio
Parts:
- J3: footprint (none) -> Socket_Strips:Socket_Strip_Straight_1x04_Pitch2.54mm
- TP21, TP22: footprint (none) -> footprints:TestPoint_THTPad_D1.5mm_Drill0.7mm
Changed lines of the file:
@@
 F 0 "J3" H 5150 4100 50  0000 C CNN
 F 1 "Conn_01x04" H 5150 3600 50  0000 C CNN
-F 2 "" H 5150 3900 50  0001 C CNN
+F 2 "Socket_Strips:Socket_Strip_Straight_1x04_Pitch2.54mm" H 5150 3900 50  0001 C CNN
 F 3 "" H 5150 3900 50  0001 C CNN
 	1    5150 3900
@@
 $EndComp
 $Comp
-L GND #PWR22
+L GND #PWR022
 U 1 1 5B96559F
 P 5600 4600
-F 0 "#PWR22" H 5600 4350 50  0001 C CNN
+F 0 "#PWR022" H 5600 4350 50  0001 C CNN
 F 1 "GND" H 5600 4450 50  0000 C CNN
 F 2 "" H 5600 4600 50  0001 C CNN
@@
 $EndComp
 $Comp
-L +5V #PWR23
+L +5V #PWR023
 U 1 1 5B9655B5
 P 5800 3450
-F 0 "#PWR23" H 5800 3300 50  0001 C CNN
+F 0 "#PWR023" H 5800 3300 50  0001 C CNN
 F 1 "+5V" H 5800 3590 50  0000 C CNN
 F 2 "" H 5800 3450 50  0001 C CNN
@@
 $EndComp
 $Comp
-L +3V3 #PWR24
+L +3V3 #PWR024
 U 1 1 5B9655CB
 P 6850 3450
-F 0 "#PWR24" H 6850 3300 50  0001 C CNN
+F 0 "#PWR024" H 6850 3300 50  0001 C CNN
 F 1 "+3V3" H 6850 3590 50  0000 C CNN
 F 2 "" H 6850 3450 50  0001 C CNN
@@
 $EndComp
 $Comp
-L PWR_FLAG #FLG1
+L PWR_FLAG #FLG025
 U 1 1 5B9655E1
 P 6050 3650
-F 0 "#FLG1" H 6050 3725 50  0001 C CNN
+F 0 "#FLG025" H 6050 3725 50  0001 C CNN
 F 1 "PWR_FLAG" H 6050 3800 50  0000 C CNN
 F 2 "" H 6050 3650 50  0001 C CNN
@@
 $EndComp
 $Comp
-L PWR_FLAG #FLG3
+L PWR_FLAG #FLG026
 U 1 1 5B965604
 P 7200 3850
-F 0 "#FLG3" H 7200 3925 50  0001 C CNN
+F 0 "#FLG026" H 7200 3925 50  0001 C CNN
 F 1 "PWR_FLAG" H 7200 4000 50  0000 C CNN
 F 2 "" H 7200 3850 50  0001 C CNN
@@
 $EndComp
 $Comp
-L PWR_FLAG #FLG2
+L PWR_FLAG #FLG027
 U 1 1 5B96561A
 P 6050 4300
-F 0 "#FLG2" H 6050 4375 50  0001 C CNN
+F 0 "#FLG027" H 6050 4375 50  0001 C CNN
 F 1 "PWR_FLAG" H 6050 4450 50  0000 C CNN
 F 2 "" H 6050 4300 50  0001 C CNN
@@
 F 0 "TP21" H 6350 4050 50  0000 C BNN
 F 1 "TEST" H 6350 4000 50  0000 C CNN
-F 2 "" H 6350 3750 50  0001 C CNN
+F 2 "footprints:TestPoint_THTPad_D1.5mm_Drill0.7mm" H 6350 3750 50  0001 C CNN
 F 3 "" H 6350 3750 50  0001 C CNN
 	1    6350 3750
@@
 F 0 "TP22" H 7500 4250 50  0000 C BNN
 F 1 "TEST" H 7500 4200 50  0000 C CNN
-F 2 "" H 7500 3950 50  0001 C CNN
+F 2 "footprints:TestPoint_THTPad_D1.5mm_Drill0.7mm" H 7500 3950 50  0001 C CNN
 F 3 "" H 7500 3950 50  0001 C CNN
 	1    7500 3950

Commit message: pbase edits
Parts:
- TP21: value TEST -> 5V
- TP22: value TEST -> 3V3
Changed lines of the file:
@@
 P 6350 3750
 F 0 "TP21" H 6350 4050 50  0000 C BNN
-F 1 "TEST" H 6350 4000 50  0000 C CNN
+F 1 "5V" H 6350 4000 50  0000 C CNN
 F 2 "footprints:TestPoint_THTPad_D1.5mm_Drill0.7mm" H 6350 3750 50  0001 C CNN
 F 3 "" H 6350 3750 50  0001 C CNN
@@
 P 7500 3950
 F 0 "TP22" H 7500 4250 50  0000 C BNN
-F 1 "TEST" H 7500 4200 50  0000 C CNN
+F 1 "3V3" H 7500 4200 50  0000 C CNN
 F 2 "footprints:TestPoint_THTPad_D1.5mm_Drill0.7mm" H 7500 3950 50  0001 C CNN
 F 3 "" H 7500 3950 50  0001 C CNN

Commit message: pcb fin 1
Parts:
- removed TP21: 5V, footprints:TestPoint_THTPad_D1.5mm_Drill0.7mm, symbol TEST
- removed TP22: 3V3, footprints:TestPoint_THTPad_D1.5mm_Drill0.7mm, symbol TEST
Changed lines of the file:
@@
 Connection ~ 5600 3900
 Connection ~ 5600 4500
-Wire Wire Line
-	5350 3800 6350 3800
 Connection ~ 5800 3800
-Wire Wire Line
-	5350 4000 7500 4000
 Connection ~ 6850 4000
-$Comp
-L TEST TP21
-U 1 1 5B982DEF
-P 6350 3750
-F 0 "TP21" H 6350 4050 50  0000 C BNN
-F 1 "5V" H 6350 4000 50  0000 C CNN
-F 2 "footprints:TestPoint_THTPad_D1.5mm_Drill0.7mm" H 6350 3750 50  0001 C CNN
-F 3 "" H 6350 3750 50  0001 C CNN
-	1    6350 3750
-	1    0    0    -1
-$EndComp
-$Comp
-L TEST TP22
-U 1 1 5B982E1A
-P 7500 3950
-F 0 "TP22" H 7500 4250 50  0000 C BNN
-F 1 "3V3" H 7500 4200 50  0000 C CNN
-F 2 "footprints:TestPoint_THTPad_D1.5mm_Drill0.7mm" H 7500 3950 50  0001 C CNN
-F 3 "" H 7500 3950 50  0001 C CNN
-	1    7500 3950
-	1    0    0    -1
-$EndComp
-Wire Wire Line
-	7500 4000 7500 3950
 Connection ~ 7200 4000
-Wire Wire Line
-	6350 3800 6350 3750
 Connection ~ 6050 3800
 Wire Wire Line
 	6050 4500 5600 4500
+Wire Wire Line
+	6050 3800 5350 3800
+Wire Wire Line
+	7200 4000 5350 4000
 $EndSCHEMATC

Commit message: pdfs realizados
Other:
- note added: "3v3:\n- Microcontrolador. LPCXpresspo LPC1769 \n- Comunicación inalámbrica. XBEE / XBEE PRO\n- Tarjeta SD\n\n5V:\n- GPS. EM506\n- ACELERÓMETRO. MPU9250\n- Display OLED"
- note added: "5V & 3.3V CC"
- moved on the sheet: J3
Changed lines of the file:
@@
 encoding utf-8
 Sheet 8 8
-Title "Alimentación"
-Date "2018-09-10"
+Title "Diagrama de bloques "
+Date "2018-10-30"
 Rev "A"
 Comp "UTN - FRBA"
-Comment1 ""
+Comment1 "Autores: Alegre M. E., Bautista L., Tarazona L."
 Comment2 ""
-Comment3 ""
-Comment4 ""
+Comment3 "Conectar a 5V y a 3.3V de continua."
+Comment4 "Alimentación externa de la placa."
 $EndDescr
-Text Notes 5400 3050 0    60   ~ 12
+Text Notes 5100 2000 0    157  ~ 31
 Alimentación\n
 $Comp
 L Conn_01x04 J3
 U 1 1 5B96555C
-P 5150 3900
-F 0 "J3" H 5150 4100 50  0000 C CNN
-F 1 "Conn_01x04" H 5150 3600 50  0000 C CNN
-F 2 "Socket_Strips:Socket_Strip_Straight_1x04_Pitch2.54mm" H 5150 3900 50  0001 C CNN
-F 3 "" H 5150 3900 50  0001 C CNN
-	1    5150 3900
+P 4950 3700
+F 0 "J3" H 4950 3900 50  0000 C CNN
+F 1 "Conn_01x04" H 4950 3400 50  0000 C CNN
+F 2 "Socket_Strips:Socket_Strip_Straight_1x04_Pitch2.54mm" H 4950 3700 50  0001 C CNN
+F 3 "" H 4950 3700 50  0001 C CNN
+	1    4950 3700
 	-1   0    0    1
 $EndComp
@@
 L GND #PWR022
 U 1 1 5B96559F
-P 5600 4600
-F 0 "#PWR022" H 5600 4350 50  0001 C CNN
-F 1 "GND" H 5600 4450 50  0000 C CNN
-F 2 "" H 5600 4600 50  0001 C CNN
-F 3 "" H 5600 4600 50  0001 C CNN
-	1    5600 4600
+P 5400 4400
+F 0 "#PWR022" H 5400 4150 50  0001 C CNN
+F 1 "GND" H 5400 4250 50  0000 C CNN
+F 2 "" H 5400 4400 50  0001 C CNN
+F 3 "" H 5400 4400 50  0001 C CNN
+	1    5400 4400
 	1    0    0    -1
 $EndComp
@@
 L +5V #PWR023
 U 1 1 5B9655B5
-P 5800 3450
-F 0 "#PWR023" H 5800 3300 50  0001 C CNN
-F 1 "+5V" H 5800 3590 50  0000 C CNN
-F 2 "" H 5800 3450 50  0001 C CNN
-F 3 "" H 5800 3450 50  0001 C CNN
-	1    5800 3450
+P 5600 3250
+F 0 "#PWR023" H 5600 3100 50  0001 C CNN
+F 1 "+5V" H 5600 3390 50  0000 C CNN
+F 2 "" H 5600 3250 50  0001 C CNN
+F 3 "" H 5600 3250 50  0001 C CNN
+	1    5600 3250
 	1    0    0    -1
 $EndComp
@@
 L +3V3 #PWR024
 U 1 1 5B9655CB
-P 6850 3450
-F 0 "#PWR024" H 6850 3300 50  0001 C CNN
-F 1 "+3V3" H 6850 3590 50  0000 C CNN
-F 2 "" H 6850 3450 50  0001 C CNN
-F 3 "" H 6850 3450 50  0001 C CNN
-	1    6850 3450
+P 6650 3250
+F 0 "#PWR024" H 6650 3100 50  0001 C CNN
+F 1 "+3V3" H 6650 3390 50  0000 C CNN
+F 2 "" H 6650 3250 50  0001 C CNN
+F 3 "" H 6650 3250 50  0001 C CNN
+	1    6650 3250
 	1    0    0    -1
 $EndComp
@@
 L PWR_FLAG #FLG025
 U 1 1 5B9655E1
-P 6050 3650
-F 0 "#FLG025" H 6050 3725 50  0001 C CNN
-F 1 "PWR_FLAG" H 6050 3800 50  0000 C CNN
-F 2 "" H 6050 3650 50  0001 C CNN
-F 3 "" H 6050 3650 50  0001 C CNN
-	1    6050 3650
+P 5850 3450
+F 0 "#FLG025" H 5850 3525 50  0001 C CNN
+F 1 "PWR_FLAG" H 5850 3600 50  0000 C CNN
+F 2 "" H 5850 3450 50  0001 C CNN
+F 3 "" H 5850 3450 50  0001 C CNN
+	1    5850 3450
 	1    0    0    -1
 $EndComp
@@
 L PWR_FLAG #FLG026
 U 1 1 5B965604
-P 7200 3850
-F 0 "#FLG026" H 7200 3925 50  0001 C CNN
-F 1 "PWR_FLAG" H 7200 4000 50  0000 C CNN
-F 2 "" H 7200 3850 50  0001 C CNN
-F 3 "" H 7200 3850 50  0001 C CNN
-	1    7200 3850
+P 7000 3650
+F 0 "#FLG026" H 7000 3725 50  0001 C CNN
+F 1 "PWR_FLAG" H 7000 3800 50  0000 C CNN
+F 2 "" H 7000 3650 50  0001 C CNN
+F 3 "" H 7000 3650 50  0001 C CNN
+	1    7000 3650
 	1    0    0    -1
 $EndComp
@@
 L PWR_FLAG #FLG027
 U 1 1 5B96561A
-P 6050 4300
-F 0 "#FLG027" H 6050 4375 50  0001 C CNN
-F 1 "PWR_FLAG" H 6050 4450 50  0000 C CNN
-F 2 "" H 6050 4300 50  0001 C CNN
-F 3 "" H 6050 4300 50  0001 C CNN
-	1    6050 4300
+P 5850 4100
+F 0 "#FLG027" H 5850 4175 50  0001 C CNN
+F 1 "PWR_FLAG" H 5850 4250 50  0000 C CNN
+F 2 "" H 5850 4100 50  0001 C CNN
+F 3 "" H 5850 4100 50  0001 C CNN
+	1    5850 4100
 	1    0    0    -1
 $EndComp
 Wire Wire Line
-	6850 3450 6850 4000
+	6650 3250 6650 3800
 Wire Wire Line
-	5800 3800 5800 3450
+	5600 3600 5600 3250
 Wire Wire Line
-	6050 3800 6050 3650
+	5850 3600 5850 3450
 Wire Wire Line
-	7200 4000 7200 3850
+	7000 3800 7000 3650
 Wire Wire Line
-	6050 4500 6050 4300
+	5850 4300 5850 4100
 Wire Wire Line
-	5350 3700 5600 3700
+	5150 3500 5400 3500
 Wire Wire Line
-	5600 3700 5600 4600
+	5400 3500 5400 4400
 Wire Wire Line
-	5350 3900 5600 3900
-Connection ~ 5600 3900
-Connection ~ 5600 4500
-Connection ~ 5800 3800
-Connection ~ 6850 4000
-Connection ~ 7200 4000
-Connection ~ 6050 3800
+	5150 3700 5400 3700
+Connection ~ 5400 3700
+Connection ~ 5400 4300
+Connection ~ 5600 3600
+Connection ~ 6650 3800
+Connection ~ 7000 3800
+Connection ~ 5850 3600
 Wire Wire Line
-	6050 4500 5600 4500
+	5850 4300 5400 4300
 Wire Wire Line
-	6050 3800 5350 3800
+	5850 3600 5150 3600
 Wire Wire Line
-	7200 4000 5350 4000
+	7000 3800 5150 3800
+Text Notes 5450 2300 0    79   ~ 0
+5V & 3.3V CC
+Text Notes 1200 7450 0    79   ~ 0
+3v3:\n- Microcontrolador. LPCXpresspo LPC1769 \n- Comunicación inalámbrica. XBEE / XBEE PRO\n- Tarjeta SD\n\n5V:\n- GPS. EM506\n- ACELERÓMETRO. MPU9250\n- Display OLED
+Wire Notes Line
+	1100 6250 1100 7550
+Wire Notes Line
+	1100 7550 4200 7550
+Wire Notes Line
+	4200 7550 4200 6250
+Wire Notes Line
+	4200 6250 1100 6250
 $EndSCHEMATC
