File: pcbs/pbase/GPS.sch (KiCad schematic (older format))
At the start: 1 part

Commit message: sch annotate v1.1
Parts:
- gave numbers to parts that had none: 1
Changed lines of the file:
@@
 $EndDescr
 $Comp
-L GPS_EM506 U?
+L GPS_EM506 U3
 U 1 1 5B961160
 P 5500 3700
-F 0 "U?" H 6200 3750 60  0000 C CNN
+F 0 "U3" H 6200 3750 60  0000 C CNN
 F 1 "GPS_EM506" H 5750 3750 60  0000 C CNN
 F 2 "" H 5500 3700 60  0001 C CNN
@@
 $EndComp
 $Comp
-L GND #PWR011
+L GND #PWR12
 U 1 1 5B9611FC
 P 5900 4500
-F 0 "#PWR011" H 5900 4250 50  0001 C CNN
+F 0 "#PWR12" H 5900 4250 50  0001 C CNN
 F 1 "GND" H 5900 4350 50  0000 C CNN
 F 2 "" H 5900 4500 50  0001 C CNN
@@
 $EndComp
 $Comp
-L +5V #PWR012
+L +5V #PWR11
 U 1 1 5B961212
 P 5200 3500
-F 0 "#PWR012" H 5200 3350 50  0001 C CNN
+F 0 "#PWR11" H 5200 3350 50  0001 C CNN
 F 1 "+5V" H 5200 3640 50  0000 C CNN
 F 2 "" H 5200 3500 50  0001 C CNN

Commit message: pbase pcb inicio
Parts:
- U3: footprint (none) -> Connectors_JST:JST_SH_SM06B-SRSS-TB_06x1.00mm_Angled
Changed lines of the file:
@@
 F 0 "U3" H 6200 3750 60  0000 C CNN
 F 1 "GPS_EM506" H 5750 3750 60  0000 C CNN
-F 2 "" H 5500 3700 60  0001 C CNN
+F 2 "Connectors_JST:JST_SH_SM06B-SRSS-TB_06x1.00mm_Angled" H 5500 3700 60  0001 C CNN
 F 3 "" H 5500 3700 60  0001 C CNN
 	1    5500 3700
@@
 $EndComp
 $Comp
-L GND #PWR12
+L GND #PWR011
 U 1 1 5B9611FC
 P 5900 4500
-F 0 "#PWR12" H 5900 4250 50  0001 C CNN
+F 0 "#PWR011" H 5900 4250 50  0001 C CNN
 F 1 "GND" H 5900 4350 50  0000 C CNN
 F 2 "" H 5900 4500 50  0001 C CNN
@@
 $EndComp
 $Comp
-L +5V #PWR11
+L +5V #PWR012
 U 1 1 5B961212
 P 5200 3500
-F 0 "#PWR11" H 5200 3350 50  0001 C CNN
+F 0 "#PWR012" H 5200 3350 50  0001 C CNN
 F 1 "+5V" H 5200 3640 50  0000 C CNN
 F 2 "" H 5200 3500 50  0001 C CNN

Commit message: pdfs de pcbs finalizados. Contienen SCH, PCB y BOM.
Other:
- note added: "EM506"
- note added: "GPS"
- note removed: "GPS\n"
Changed lines of the file:
@@
 Rev "A"
 Comp "UTN - FRBA"
-Comment1 ""
+Comment1 "Autores: Alegre M. E., Bautista L., Tarazona L."
 Comment2 ""
 Comment3 "Antena incorporada. 30x30 mm. Largo cable 30mm. UART."
@@
 Text HLabel 5200 3900 0    60   Input ~ 0
 TXD3
-Text Notes 5800 3250 0    60   ~ 12
-GPS\n
+Text Notes 5650 2650 0    157  ~ 31
+GPS
+Text Notes 5750 2850 0    60   ~ 0
+EM506
 $EndSCHEMATC
