File: pcbs/pbase-ino/GPS.sch (KiCad schematic (older format))
At the start: 1 part, among them U3 GPS_EM506

Commit message: pdfs realizados
Other:
- note added: "EM-506"
Changed lines of the file:
@@
 encoding utf-8
 Sheet 3 7
-Title "GPS"
-Date "2018-09-10"
+Title "TAUTOLOGICAL"
+Date "2018-10-30"
 Rev "A"
-Comp "UTN - FRBA"
-Comment1 ""
-Comment2 ""
-Comment3 ""
-Comment4 ""
+Comp "UTN-FRBA"
+Comment1 "Autores: Alegre M. E., Bautista L., Tarazona L."
+Comment2 "Antena incorporada. 30x30 mm. Largo cable 30mm. UART."
+Comment3 "GPS EM506"
+Comment4 "Sport Tracker."
 $EndDescr
 $Comp
@@
 Text HLabel 5200 3900 0    60   Input ~ 0
 TXD3
-Text Notes 5800 3250 0    60   ~ 12
+Text Notes 5650 2650 0    157  ~ 31
 GPS\n
+Text Notes 5650 2900 0    79   ~ 16
+EM-506
 $EndSCHEMATC
