File: pcbs/pbase-ino/TarjetaSD.sch (KiCad schematic (older format))
At the start: 11 parts, among them J1 SD_Card

Commit message: PCBs pbase y pbase-ino FINALIZADOS, archivos gerbers en zip dentro del directrio /pcbs
Parts:
- J1: footprint Connectors:SD_Card_Receptacle -> footprints:SD_TE_2041021_edit
Connections:
- net +3V3: now also R2.1, R3.1
- net +5V: no longer R2.1, R3.1
Changed lines of the file:
@@
 F 0 "J1" H 4800 2750 50  0000 C CNN
 F 1 "SD_Card" H 6050 1650 50  0000 C CNN
-F 2 "Connectors:SD_Card_Receptacle" H 5650 2550 50  0001 C CNN
+F 2 "footprints:SD_TE_2041021_edit" H 5650 2550 50  0001 C CNN
 F 3 "" H 5450 2200 50  0001 C CNN
 	1    5450 2200
@@
 	4550 2600 4300 2600
 Wire Wire Line
-	4750 3450 6550 3450
-Wire Wire Line
 	6550 3450 6550 3350
 Wire Wire Line
 	5550 3550 5550 3450
-Connection ~ 5550 3450
 Wire Wire Line
 	5950 3550 5950 3450
@@
 	4350 4400 6650 4400
 Wire Wire Line
-	6350 3550 6350 3450
+	6350 3450 6350 3550
 Connection ~ 6350 3450
 Wire Wire Line
@@
 Wire Wire Line
 	5550 4800 5550 4950
-Connection ~ 5150 3450
-Wire Wire Line
-	5150 3550 5150 3450
 Wire Wire Line
 	4750 3550 4750 3450
@@
 Text Notes 6700 3450 0    60   ~ 0
 -> Tensión con la que el microcontrolador maneja SPI!\n+5V arduino\n+3v3 lpc1769
+Wire Wire Line
+	5150 3450 5150 3550
+Wire Wire Line
+	5550 3450 6550 3450
+$Comp
+L +3V3 #PWR020
+U 1 1 5BB2A1E8
+P 4950 3350
+F 0 "#PWR020" H 4950 3200 50  0001 C CNN
+F 1 "+3V3" H 4950 3490 50  0000 C CNN
+F 2 "" H 4950 3350 50  0001 C CNN
+F 3 "" H 4950 3350 50  0001 C CNN
+	1    4950 3350
+	1    0    0    -1
+$EndComp
+Wire Wire Line
+	4750 3450 5150 3450
+Wire Wire Line
+	4950 3450 4950 3350
+Connection ~ 4950 3450
 $EndSCHEMATC

Commit message: pdfs realizados
Other:
- note added: "En este caso, seguir estas especificaciones para conectarla al arduino."
- note added: "IMPORTANTE:\nConexionado basado en el siguiente tutorial: https://www.youtube.com/watch?v=E7l2UUhi0jk&t=249s\n\nSegún el mismo, para ARDUINO, los valores de los resistores son los siguientes:\n- R2 y R3 No se conectan.\n- R4 = R5 = R6 = 1K8\n- R7 = R8 = R9 = 3K3\n\nSegún kit infotronic, para LPC1769:\n- R2 = R3 = 10K\n- R4 = R5 = 33K\n- R6, R7, R8 Y R9 NO SE CONECTAN\n----------------------------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"
- note removed: "IMPORTANTE:\nConexionado basado en el siguiente tutorial: https://www.youtube.com/watch?v=E7l2UUhi0jk&t=249s\n\nSegún el mismo, los valores de los resistores son los siguientes:\nR2 y R3 No se conectan.\nR4 = R5=R6 = 1K8\nR7=R8=R9 = 3K3\n\nSegún kit infotronic:\nR2 = R3 = 10K\nR4 = R5 = 33K\nR6, R7, R8 Y R9 NO SE CONECTAN\n----------------------------------------------------------------\nEsto ocu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"
- moved on the sheet: C1, C2, J1, R2, R3, R4, R5, R6, R7, R8, R9
