File: pcbs/pbase-ino/Zigbee.sch (KiCad schematic (older format))
At the start: 1 part

Commit message: pdfs realizados
Other:
- note added: "Comunicación inalámbrica - Zigbee"
- note added: "XBEE / XBEE-PRO"
- note removed: "Comunicación Zigbee"
Changed lines of the file:
@@
 encoding utf-8
 Sheet 5 7
-Title "Zigbee"
-Date "2018-09-10"
+Title "TAUTOLOGICAL"
+Date "2018-10-30"
 Rev "A"
-Comp "UTN - FRBA"
-Comment1 ""
+Comp "UTN-FRBA"
+Comment1 "Autores: Alegre M. E., Bautista L., Tarazona L."
 Comment2 ""
-Comment3 ""
-Comment4 ""
+Comment3 "Antena incorporada. UART."
+Comment4 "Comunicación Zigbee. XBEE / XBEE-PRO"
 $EndDescr
 $Comp
@@
 	7600 3750 8100 3750
 Wire Wire Line
-	7600 3950 8100 3950
+	7600 3850 8100 3850
 Text Label 7600 3450 2    60   ~ 0
 RXD1
@@
 Text Label 7600 3750 2    60   ~ 0
 SLEEP
-Text Label 7600 3950 2    60   ~ 0
+Text Label 7600 3850 2    60   ~ 0
 RSSI
 Text HLabel 8100 3450 2    60   Output ~ 0
@@
 Text HLabel 8100 3750 2    60   Output ~ 0
 SLEEP
-Text HLabel 8100 3950 2    60   Output ~ 0
+Text HLabel 8100 3850 2    60   Output ~ 0
 RSSI
 $Comp
@@
 	1    0    0    -1
 $EndComp
-Text Notes 5300 2650 0    60   ~ 12
-Comunicación Zigbee
+Text Notes 3700 1700 0    157  ~ 31
+Comunicación inalámbrica - Zigbee
 NoConn ~ 6550 3950
 NoConn ~ 6550 4250
+Text Notes 5200 2050 0    79   ~ 16
+XBEE / XBEE-PRO
 $EndSCHEMATC
