File: pcbs/pbase-ino/acc.sch (KiCad schematic (older format))
At the start: 2 parts, among them U2 acc_mpu9250_board

Commit message: pdfs realizados
Other:
- note added: "- Módulo acelerómetro MPU 9250.\n- El mismo consta con un acelerómetro, un giróscopo y un magnetómetro.\n- Información en los tres ejes X,Y,Z.\n- A travéz del pin 7 (ADO) puede modificarse su dirección llevándolo a VCC (5v).\n- R1 es un jumper. Quitarlo si se desea conservar la dirección que trae por defecto.\n- Si FSYNC no se usa ponerlo a GND o en LOW.\n- Cuenta con un regulador interno low dro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"
- note added: "En este caso, soldarlo o no, no trae complicación alguna."
- note added: "mpu9250"
Changed lines of the file:
@@
 encoding utf-8
 Sheet 2 7
-Title "Acelerómetro"
-Date "2018-09-10"
+Title "TAUTOLOGICAL"
+Date "2018-10-30"
 Rev "A"
-Comp "UTN - FRBA"
-Comment1 "Si FSYNC no se usa ponerlo a GND o en LOW."
-Comment2 "R1 es un jumper. Quitarlo si se desea conservar la dirección que trae por defecto."
-Comment3 "Misma conexión que el MPU6050."
-Comment4 "Este acelerómetro ya incorpora un magnetómetro."
+Comp "UTN-FRBA"
+Comment1 "Autores: Alegre M. E., Bautista L., Tarazona L."
+Comment2 ""
+Comment3 "Pin [1:8] compatible con MPU6050."
+Comment4 "Acelerómetro MPU9250. con magnetómetro. I2C."
 $EndDescr
 $Comp
@@
 Text HLabel 5600 3650 0    60   BiDi ~ 0
 SCL0
-Text Notes 5800 2800 0    60   ~ 12
+Text Notes 5100 1950 0    157  ~ 31
 Acelerómetro
-Wire Wire Line
-	5800 3650 5600 3650
-Wire Wire Line
-	5800 3750 5600 3750
-Wire Wire Line
-	5800 4150 5600 4150
-Wire Wire Line
-	5800 3450 5600 3450
-Wire Wire Line
-	5600 3450 5600 3250
-Wire Wire Line
-	5800 3550 5050 3550
-Wire Wire Line
-	5050 3550 5050 3650
 $Comp
 L R R1
@@
 	1    0    0    -1
 $EndComp
-Wire Wire Line
-	5800 4050 4700 4050
-Wire Wire Line
-	4700 4050 4700 3900
-Wire Wire Line
-	4700 3600 4700 3250
 $Comp
 L +5V #PWR03
@@
 Text HLabel 5600 4350 0    60   Input ~ 0
 FSYNC
+Text Notes 1150 7600 0    79   ~ 16
+- Módulo acelerómetro MPU 9250.\n- El mismo consta con un acelerómetro, un giróscopo y un magnetómetro.\n- Información en los tres ejes X,Y,Z.\n- A travéz del pin 7 (ADO) puede modificarse su dirección llevándolo a VCC (5v).\n- R1 es un jumper. Quitarlo si se desea conservar la dirección que trae por defecto.\n- Si FSYNC no se usa ponerlo a GND o en LOW.\n- Cuenta con un regulador interno low dropout de 3v3 para conectarse a 5v.\nPor lo que puede conectarse tanto a 5V como a 3V3.
+Text Notes 5600 2150 0    79   ~ 16
+mpu9250
+Wire Wire Line
+	5800 3650 5600 3650
+Wire Wire Line
+	5800 3750 5600 3750
+Wire Wire Line
+	5800 4150 5600 4150
+Wire Wire Line
+	5800 3450 5600 3450
+Wire Wire Line
+	5600 3450 5600 3250
+Wire Wire Line
+	5800 3550 5050 3550
+Wire Wire Line
+	5050 3550 5050 3650
+Wire Wire Line
+	5800 4050 4700 4050
+Wire Wire Line
+	4700 4050 4700 3900
+Wire Wire Line
+	4700 3600 4700 3250
 Wire Wire Line
 	5600 4350 5800 4350
+Wire Notes Line
+	1050 6400 1050 7700
+Wire Notes Line
+	1050 7700 6550 7700
+Wire Notes Line
+	6550 7700 6550 6400
+Wire Notes Line
+	6550 6400 1050 6400
+Text Notes 1100 4500 0    79   ~ 0
+En este caso, soldarlo o no, no trae complicación alguna.
+Wire Notes Line
+	4500 3750 4050 3750
+Wire Notes Line
+	4050 3750 3800 4150
+Wire Notes Line
+	4450 3700 4500 3750
+Wire Notes Line
+	4500 3750 4450 3800
 $EndSCHEMATC
