File: pcbs/pbase-ino/arduino-MEGA.sch (KiCad schematic (older format))
At the start: 17 parts

Commit message: PCBs pbase y pbase-ino FINALIZADOS, archivos gerbers en zip dentro del directrio /pcbs
Parts:
- TP1, TP10, TP11, TP12, TP13, TP14, TP15, TP16, TP2, TP3, TP4, TP5, TP6, TP7, TP8, TP9: footprint (none) -> footprints:TestPoint_THTPad_D1.5mm_Drill0.7mm
- XA1: footprint (none) -> footprints:Arduino_Mega2560_Shield_flippedONtop
Changed lines of the file:
@@
 F 0 "XA1" V 3850 4000 60  0000 C CNN
 F 1 "Arduino_Mega2560_Shield" V 3650 4000 60  0000 C CNN
-F 2 "" H 4450 6750 60  0001 C CNN
+F 2 "footprints:Arduino_Mega2560_Shield_flippedONtop" H 4450 6750 60  0001 C CNN
 F 3 "" H 4450 6750 60  0001 C CNN
 	1    3750 4000
@@
 SCK1
 $Comp
-L GND #PWR020
+L GND #PWR021
 U 1 1 5BB16AB6
 P 2050 5500
-F 0 "#PWR020" H 2050 5250 50  0001 C CNN
+F 0 "#PWR021" H 2050 5250 50  0001 C CNN
 F 1 "GND" H 2050 5350 50  0000 C CNN
 F 2 "" H 2050 5500 50  0001 C CNN
@@
 $EndComp
 $Comp
-L +5V #PWR021
+L +5V #PWR022
 U 1 1 5BB16C81
 P 1650 5800
-F 0 "#PWR021" H 1650 5650 50  0001 C CNN
+F 0 "#PWR022" H 1650 5650 50  0001 C CNN
 F 1 "+5V" H 1650 5940 50  0000 C CNN
 F 2 "" H 1650 5800 50  0001 C CNN
@@
 $EndComp
 $Comp
-L GND #PWR022
+L GND #PWR023
 U 1 1 5BB16F14
 P 4250 1300
-F 0 "#PWR022" H 4250 1050 50  0001 C CNN
+F 0 "#PWR023" H 4250 1050 50  0001 C CNN
 F 1 "GND" H 4250 1150 50  0000 C CNN
 F 2 "" H 4250 1300 50  0001 C CNN
@@
 $EndComp
 $Comp
-L +5V #PWR023
+L +5V #PWR024
 U 1 1 5BB1716A
 P 3800 1050
-F 0 "#PWR023" H 3800 900 50  0001 C CNN
+F 0 "#PWR024" H 3800 900 50  0001 C CNN
 F 1 "+5V" H 3800 1190 50  0000 C CNN
 F 2 "" H 3800 1050 50  0001 C CNN
@@
 F 0 "TP1" H 8100 2200 50  0000 C BNN
 F 1 "SDA0" H 8100 2150 50  0000 C CNN
-F 2 "" H 8100 1900 50  0001 C CNN
+F 2 "footprints:TestPoint_THTPad_D1.5mm_Drill0.7mm" H 8100 1900 50  0001 C CNN
 F 3 "" H 8100 1900 50  0001 C CNN
 	1    8100 1900
@@
 F 0 "TP2" H 8300 2200 50  0000 C BNN
 F 1 "SCL0" H 8300 2150 50  0000 C CNN
-F 2 "" H 8300 1900 50  0001 C CNN
+F 2 "footprints:TestPoint_THTPad_D1.5mm_Drill0.7mm" H 8300 1900 50  0001 C CNN
 F 3 "" H 8300 1900 50  0001 C CNN
 	1    8300 1900
@@
 F 0 "TP3" H 8500 2200 50  0000 C BNN
 F 1 "INT" H 8500 2150 50  0000 C CNN
-F 2 "" H 8500 1900 50  0001 C CNN
+F 2 "footprints:TestPoint_THTPad_D1.5mm_Drill0.7mm" H 8500 1900 50  0001 C CNN
 F 3 "" H 8500 1900 50  0001 C CNN
 	1    8500 1900
@@
 F 0 "TP4" H 8700 2200 50  0000 C BNN
 F 1 "FSYNC" H 8700 2150 50  0000 C CNN
-F 2 "" H 8700 1900 50  0001 C CNN
+F 2 "footprints:TestPoint_THTPad_D1.5mm_Drill0.7mm" H 8700 1900 50  0001 C CNN
 F 3 "" H 8700 1900 50  0001 C CNN
 	1    8700 1900
@@
 F 0 "TP5" H 8150 3150 50  0000 C BNN
 F 1 "TXD3" H 8150 3100 50  0000 C CNN
-F 2 "" H 8150 2850 50  0001 C CNN
+F 2 "footprints:TestPoint_THTPad_D1.5mm_Drill0.7mm" H 8150 2850 50  0001 C CNN
 F 3 "" H 8150 2850 50  0001 C CNN
 	1    8150 2850
@@
 F 0 "TP6" H 8450 3150 50  0000 C BNN
 F 1 "RXD3" H 8450 3100 50  0000 C CNN
-F 2 "" H 8450 2850 50  0001 C CNN
+F 2 "footprints:TestPoint_THTPad_D1.5mm_Drill0.7mm" H 8450 2850 50  0001 C CNN
 F 3 "" H 8450 2850 50  0001 C CNN
 	1    8450 2850
@@
 F 0 "TP7" H 8750 3150 50  0000 C BNN
 F 1 "DIR" H 8750 3100 50  0000 C CNN
-F 2 "" H 8750 2850 50  0001 C CNN
+F 2 "footprints:TestPoint_THTPad_D1.5mm_Drill0.7mm" H 8750 2850 50  0001 C CNN
 F 3 "" H 8750 2850 50  0001 C CNN
 	1    8750 2850
@@
 F 0 "TP8" H 7950 4000 50  0000 C BNN
 F 1 "RXD1" H 7950 3950 50  0000 C CNN
-F 2 "" H 7950 3700 50  0001 C CNN
+F 2 "footprints:TestPoint_THTPad_D1.5mm_Drill0.7mm" H 7950 3700 50  0001 C CNN
 F 3 "" H 7950 3700 50  0001 C CNN
 	1    7950 3700
@@
 F 0 "TP9" H 8150 4000 50  0000 C BNN
 F 1 "TXD1" H 8150 3950 50  0000 C CNN
-F 2 "" H 8150 3700 50  0001 C CNN
+F 2 "footprints:TestPoint_THTPad_D1.5mm_Drill0.7mm" H 8150 3700 50  0001 C CNN
 F 3 "" H 8150 3700 50  0001 C CNN
 	1    8150 3700
@@
 F 0 "TP10" H 8400 4000 50  0000 C BNN
 F 1 "SLEEP" H 8400 3950 50  0000 C CNN
-F 2 "" H 8400 3700 50  0001 C CNN
+F 2 "footprints:TestPoint_THTPad_D1.5mm_Drill0.7mm" H 8400 3700 50  0001 C CNN
 F 3 "" H 8400 3700 50  0001 C CNN
 	1    8400 3700
@@
 F 0 "TP11" H 8650 4000 50  0000 C BNN
 F 1 "SRQ" H 8650 3950 50  0000 C CNN
-F 2 "" H 8650 3700 50  0001 C CNN
+F 2 "footprints:TestPoint_THTPad_D1.5mm_Drill0.7mm" H 8650 3700 50  0001 C CNN
 F 3 "" H 8650 3700 50  0001 C CNN
 	1    8650 3700
@@
 F 0 "TP12" H 8850 4000 50  0000 C BNN
 F 1 "CAP2" H 8850 3950 50  0000 C CNN
-F 2 "" H 8850 3700 50  0001 C CNN
+F 2 "footprints:TestPoint_THTPad_D1.5mm_Drill0.7mm" H 8850 3700 50  0001 C CNN
 F 3 "" H 8850 3700 50  0001 C CNN
 	1    8850 3700
@@
 F 0 "TP13" H 8100 5300 50  0000 C BNN
 F 1 "MOSI1" H 8100 5250 50  0000 C CNN
-F 2 "" H 8100 5000 50  0001 C CNN
+F 2 "footprints:TestPoint_THTPad_D1.5mm_Drill0.7mm" H 8100 5000 50  0001 C CNN
 F 3 "" H 8100 5000 50  0001 C CNN
 	1    8100 5000
@@
 F 0 "TP14" H 8350 5300 50  0000 C BNN
 F 1 "MISO1" H 8350 5250 50  0000 C CNN
-F 2 "" H 8350 5000 50  0001 C CNN
+F 2 "footprints:TestPoint_THTPad_D1.5mm_Drill0.7mm" H 8350 5000 50  0001 C CNN
 F 3 "" H 8350 5000 50  0001 C CNN
 	1    8350 5000
@@
 F 0 "TP15" H 8600 5300 50  0000 C BNN
 F 1 "SCK1" H 8600 5250 50  0000 C CNN
-F 2 "" H 8600 5000 50  0001 C CNN
+F 2 "footprints:TestPoint_THTPad_D1.5mm_Drill0.7mm" H 8600 5000 50  0001 C CNN
 F 3 "" H 8600 5000 50  0001 C CNN
 	1    8600 5000
@@
 F 0 "TP16" H 8850 5300 50  0000 C BNN
 F 1 "SSEL1" H 8850 5250 50  0000 C CNN
-F 2 "" H 8850 5000 50  0001 C CNN
+F 2 "footprints:TestPoint_THTPad_D1.5mm_Drill0.7mm" H 8850 5000 50  0001 C CNN
 F 3 "" H 8850 5000 50  0001 C CNN
 	1    8850 5000
@@
 NoConn ~ 2450 5050
 $Comp
-L PWR_FLAG #FLG024
+L PWR_FLAG #FLG025
 U 1 1 5BB2D1A8
 P 4150 1050
-F 0 "#FLG024" H 4150 1125 50  0001 C CNN
+F 0 "#FLG025" H 4150 1125 50  0001 C CNN
 F 1 "PWR_FLAG" H 4150 1200 50  0000 C CNN
 F 2 "" H 4150 1050 50  0001 C CNN

Commit message: pdfs realizados
Other:
- note added: "ARDUINO MEGA"
- note added: "MICROCONTROLADOR"
- note added: "TEST POINTS"
- moved on the sheet: TP1, TP10, TP11, TP12, TP13, TP14, TP15, TP16, TP2, TP3, TP4, TP5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
