File: pcbs/pbase-ino/pbase-ino.sch (KiCad schematic (older format))
At the start: 0 parts

Commit message: pdfs realizados
Other:
- note added: "Placa base - ino"
- note added: "TAUTOLOGICAL"
Changed lines of the file:
@@
 encoding utf-8
 Sheet 1 7
-Title ""
-Date ""
-Rev ""
-Comp ""
-Comment1 ""
-Comment2 ""
-Comment3 ""
-Comment4 ""
+Title "TAUTOLOGICAL"
+Date "2018-10-30"
+Rev "A"
+Comp "UTN-FRBA"
+Comment1 "https://github.com/ealegremendoza/proyecto_4to"
+Comment2 "Autores: Alegre M. E., Bautista L., Tarazona L."
+Comment3 "Medidor de posición y velocidad de sujetos en movimiento."
+Comment4 "Sport Tracker."
 $EndDescr
 $Sheet
-S 2700 2300 1350 750
+S 3000 2800 1350 750
 U 5BB15359
 F0 "acc" 60
 F1 "acc.sch" 60
-F2 "INT" O R 4050 2750 60
-F3 "SDA0" B R 4050 2450 60
-F4 "SCL0" B R 4050 2600 60
-F5 "FSYNC" I R 4050 2900 60
+F2 "INT" O R 4350 3250 60
+F3 "SDA0" B R 4350 2950 60
+F4 "SCL0" B R 4350 3100 60
+F5 "FSYNC" I R 4350 3400 60
 $EndSheet
 $Sheet
-S 2700 3550 1350 550
+S 3000 4050 1350 550
 U 5BB15400
 F0 "GPS" 60
 F1 "GPS.sch" 60
-F2 "DIR" O R 4050 4000 60
-F3 "RXD3" O R 4050 3850 60
-F4 "TXD3" I R 4050 3700 60
+F2 "DIR" O R 4350 4500 60
+F3 "RXD3" O R 4350 4350 60
+F4 "TXD3" I R 4350 4200 60
 $EndSheet
 $Sheet
-S 2700 4600 1350 500
+S 3000 5100 1350 500
 U 5BB15418
 F0 "Alimentación" 60
 F1 "pwr.sch" 60
-F2 "VBat" O R 4050 4850 60
+F2 "VBat" O R 4350 5350 60
 $EndSheet
 $Sheet
-S 7200 2300 1350 900
+S 7500 2800 1350 900
 U 5BB15468
 F0 "Zigbee" 60
 F1 "Zigbee.sch" 60
-F2 "RXD1" O L 7200 2600 60
-F3 "TXD1" I L 7200 2450 60
-F4 "SLRQ" I L 7200 2900 60
-F5 "SLEEP" O L 7200 2750 60
-F6 "RSSI" O L 7200 3050 60
+F2 "RXD1" O L 7500 3100 60
+F3 "TXD1" I L 7500 2950 60
+F4 "SLRQ" I L 7500 3400 60
+F5 "SLEEP" O L 7500 3250 60
+F6 "RSSI" O L 7500 3550 60
 $EndSheet
 $Sheet
-S 7200 4350 1350 800
+S 7500 4850 1350 800
 U 5BB154A3
 F0 "Tarjeta SD" 60
 F1 "TarjetaSD.sch" 60
-F2 "SSEL1" I L 7200 4950 60
-F3 "MOSI1" I L 7200 4500 60
-F4 "MISO1" O L 7200 4650 60
-F5 "SCK1" I L 7200 4800 60
+F2 "SSEL1" I L 7500 5450 60
+F3 "MOSI1" I L 7500 5000 60
+F4 "MISO1" O L 7500 5150 60
+F5 "SCK1" I L 7500 5300 60
 $EndSheet
 Wire Wire Line
-	4050 2450 4800 2450
+	4350 2950 5100 2950
 Wire Wire Line
-	4050 2600 4800 2600
+	4350 3100 5100 3100
 Wire Wire Line
-	4050 2750 4800 2750
+	4350 3250 5100 3250
 Wire Wire Line
-	4050 2900 4800 2900
+	4350 3400 5100 3400
 Wire Wire Line
-	4050 3700 4800 3700
+	4350 4200 5100 4200
 Wire Wire Line
-	4800 3850 4050 3850
+	5100 4350 4350 4350
 Wire Wire Line
-	4050 4000 4800 4000
+	4350 4500 5100 4500
 Wire Wire Line
-	4050 4850 4800 4850
+	4350 5350 5100 5350
 Wire Wire Line
-	6450 4950 7200 4950
+	6750 5450 7500 5450
 Wire Wire Line
-	7200 4800 6450 4800
+	7500 5300 6750 5300
 Wire Wire Line
-	6450 4650 7200 4650
+	6750 5150 7500 5150
 Wire Wire Line
-	7200 4500 6450 4500
+	7500 5000 6750 5000
 Wire Wire Line
-	6450 2450 7200 2450
+	6750 2950 7500 2950
 Wire Wire Line
-	7200 2600 6450 2600
+	7500 3100 6750 3100
 Wire Wire Line
-	6450 2750 7200 2750
+	6750 3250 7500 3250
 Wire Wire Line
-	7200 2900 6450 2900
+	7500 3400 6750 3400
 Wire Wire Line
-	6450 3050 7200 3050
+	6750 3550 7500 3550
 $Sheet
-S 4800 2300 1650 2850
+S 5100 2800 1650 2850
 U 5BB154FA
 F0 "Microcontrolador" 60
 F1 "arduino-MEGA.sch" 60
-F2 "Vin" I L 4800 4850 60
-F3 "INT" I L 4800 2750 60
-F4 "RXD3" I L 4800 3850 60
-F5 "DIR" I L 4800 4000 60
-F6 "SDA0" B L 4800 2450 60
-F7 "SCL0" B L 4800 2600 60
-F8 "FSYNC" O L 4800 2900 60
-F9 "TXD3" O L 4800 3700 60
-F10 "RXD1" I R 6450 2600 60
-F11 "TXD1" O R 6450 2450 60
-F12 "SLEEP" I R 6450 2750 60
-F13 "SRQ" O R 6450 2900 60
-F14 "CAP2.1" I R 6450 3050 60
-F15 "MOSI1" O R 6450 4500 60
-F16 "MISO1" I R 6450 4650 60
-F17 "SCK1" B R 6450 4800 60
-F18 "SSEL1" B R 6450 4950 60
+F2 "Vin" I L 5100 5350 60
+F3 "INT" I L 5100 3250 60
+F4 "RXD3" I L 5100 4350 60
+F5 "DIR" I L 5100 4500 60
+F6 "SDA0" B L 5100 2950 60
+F7 "SCL0" B L 5100 3100 60
+F8 "FSYNC" O L 5100 3400 60
+F9 "TXD3" O L 5100 4200 60
+F10 "RXD1" I R 6750 3100 60
+F11 "TXD1" O R 6750 2950 60
+F12 "SLEEP" I R 6750 3250 60
+F13 "SRQ" O R 6750 3400 60
+F14 "CAP2.1" I R 6750 3550 60
+F15 "MOSI1" O R 6750 5000 60
+F16 "MISO1" I R 6750 5150 60
+F17 "SCK1" B R 6750 5300 60
+F18 "SSEL1" B R 6750 5450 60
 $EndSheet
+Text Notes 5100 1950 0    157  ~ 31
+TAUTOLOGICAL
+Text Notes 5400 2150 0    79   ~ 16
+Placa base - ino
 $EndSCHEMATC
