File: pcbs/pbase-ino/pwr.sch (KiCad schematic (older format))
At the start: 9 parts, among them J2 Screw_Terminal_01x02, SW1 SW_SPDT, U1 LM2575-3.3

Commit message: PCBs pbase y pbase-ino FINALIZADOS, archivos gerbers en zip dentro del directrio /pcbs
Parts:
- removed SW1: SW_SPDT, Buttons_Switches_THT:SW_CuK_OS102011MA1QN1_SPDT_Angled, symbol SW_SPDT
- added SW1: SW_SPST, footprints:TerminalBlock_bornier-2_P5.08mm, symbol SW_SPST
- C3: footprint (none) -> Capacitors_SMD:CP_Elec_6.3x5.3
- C4: footprint (none) -> Capacitors_SMD:CP_Elec_10x10.5
- D1: footprint (none) -> Diodes_THT:D_DO-41_SOD81_P7.62mm_Horizontal
- L1: footprint (none) -> footprints:Choke_PK0810
- U1: footprint (none) -> TO_SOT_Packages_SMD:TO-263-5_TabPin3
Connections:
- net VBat: now also SW1.2 (B)
- net at J2.2 (Pin_2): now also SW1.1 (A)
- no-connect marks 1 -> 0
Other:
- moved on the sheet: J2
Changed lines of the file:
@@
 L Screw_Terminal_01x02 J2
 U 1 1 5BAFDCCC
-P 3850 3450
-F 0 "J2" H 3850 3550 50  0000 C CNN
-F 1 "Screw_Terminal_01x02" H 3850 3250 50  0000 C CNN
-F 2 "footprints:TerminalBlock_bornier-2_P5.08mm" H 3850 3450 50  0001 C CNN
-F 3 "" H 3850 3450 50  0001 C CNN
-	1    3850 3450
+P 3850 3350
+F 0 "J2" H 3850 3450 50  0000 C CNN
+F 1 "Screw_Terminal_01x02" H 3850 3150 50  0000 C CNN
+F 2 "footprints:TerminalBlock_bornier-2_P5.08mm" H 3850 3350 50  0001 C CNN
+F 3 "" H 3850 3350 50  0001 C CNN
+	1    3850 3350
 	-1   0    0    1
 $EndComp
@@
 F 0 "U1" H 6750 3600 50  0000 C CNN
 F 1 "LM2575-3.3" H 6150 3600 50  0000 C CNN
-F 2 "" H 6350 3250 50  0001 C CNN
+F 2 "TO_SOT_Packages_SMD:TO-263-5_TabPin3" H 6350 3250 50  0001 C CNN
 F 3 "" H 6350 3250 50  0001 C CNN
 	1    6350 3250
@@
 F 0 "C3" H 5625 3600 50  0000 L CNN
 F 1 "100u" H 5625 3400 50  0000 L CNN
-F 2 "" H 5638 3350 50  0001 C CNN
+F 2 "Capacitors_SMD:CP_Elec_6.3x5.3" H 5638 3350 50  0001 C CNN
 F 3 "" H 5600 3500 50  0001 C CNN
 	1    5600 3500
@@
 F 0 "D1" H 7250 3750 50  0000 C CNN
 F 1 "1N5817" H 7250 3550 50  0000 C CNN
-F 2 "" H 7250 3650 50  0001 C CNN
+F 2 "Diodes_THT:D_DO-41_SOD81_P7.62mm_Horizontal" H 7250 3650 50  0001 C CNN
 F 3 "" H 7250 3650 50  0001 C CNN
 	1    7250 3650
@@
 F 0 "L1" V 7550 3100 50  0000 C CNN
 F 1 "L_Core_Ferrite" V 7710 3100 50  0000 C CNN
-F 2 "" H 7600 3100 50  0001 C CNN
+F 2 "footprints:Choke_PK0810" H 7600 3100 50  0001 C CNN
 F 3 "" H 7600 3100 50  0001 C CNN
 	1    7600 3100
@@
 F 0 "C4" H 8025 3700 50  0000 L CNN
 F 1 "330u" H 8025 3500 50  0000 L CNN
-F 2 "" H 8038 3450 50  0001 C CNN
+F 2 "Capacitors_SMD:CP_Elec_10x10.5" H 8038 3450 50  0001 C CNN
 F 3 "" H 8000 3600 50  0001 C CNN
 	1    8000 3600
@@
 	1    0    0    -1
 $EndComp
-$Comp
-L SW_SPDT SW1
-U 1 1 5BB236DC
-P 4550 3350
-F 0 "SW1" H 4550 3520 50  0000 C CNN
-F 1 "SW_SPDT" H 4550 3150 50  0000 C CNN
-F 2 "Buttons_Switches_THT:SW_CuK_OS102011MA1QN1_SPDT_Angled" H 4550 3350 50  0001 C CNN
-F 3 "" H 4550 3350 50  0001 C CNN
-	1    4550 3350
-	1    0    0    -1
-$EndComp
-NoConn ~ 4750 3450
 Wire Wire Line
 	6900 3100 7450 3100
@@
 Connection ~ 4900 3250
 Wire Wire Line
-	4050 3350 4350 3350
+	4050 3250 4350 3250
 Wire Wire Line
-	4050 3450 4100 3450
+	4050 3350 4100 3350
 Wire Wire Line
-	4100 3450 4100 4000
+	4100 3350 4100 4000
 Connection ~ 4100 4000
+$Comp
+L SW_SPST SW1
+U 1 1 5BB28518
+P 4550 3250
+F 0 "SW1" H 4550 3375 50  0000 C CNN
+F 1 "SW_SPST" H 4550 3150 50  0000 C CNN
+F 2 "footprints:TerminalBlock_bornier-2_P5.08mm" H 4550 3250 50  0001 C CNN
+F 3 "" H 4550 3250 50  0001 C CNN
+	1    4550 3250
+	1    0    0    -1
+$EndComp
 $EndSCHEMATC

Commit message: pdfs realizados
Other:
- note added: "3V3:\n- Tarjeta SD\n- Comunicación Inalámbrica Zigbee.\nVBAT:\n- Arduino MEGA\n 5v:\n - GPS. EM506.\n - Acelerómetro. MPU9250."
- note added: "Fuente Switching 3v3"
- note added: "IMPORTANTE:\nC3, D1 y C4 lo mas cerca posible del puerto y GND."
- note removed: "C3, D1 y C4 lo mas cerca posible del puerto y GND"
- moved on the sheet: C3, C4, D1, J2, L1, SW1, TP21, TP22, U1
