File: pcbs/pbase-ino/pbase-ino.kicad_pcb (KiCad board)
At the start: 2 copper layers, 100 x 100 mm, 52 parts, among them J1 SD_Card, J2 Screw_Terminal_01x02, M3 MountingHole_3.2mm_M3_DIN965, SW1 SW_SPST, U1 LM2575-3.3, U2 acc_mpu9250_board, U3 GPS_EM506

Commit message: pdfs realizados
Other:
- board text added: "!"
- board text added: "330uH"
- board text added: "IMPORTANTE. - El ARDUINO MEGA va conectado al revés, boca abajo. Deben soldarse tira de pines macho. En los 6 pines centrales de este deben soldarse pines hembra. - Todos los resistores y C2 son 0805. |C1: CP_Tantalum_Case-A_EIA-3216-18. C4: CP_Elec_10x10.5. | C3:CP_Elec_6.3x5.3 - Conector del GPS: JST_SH_SM06B-SRSS-TB_06x1.00mm_Angled. - Tarjeta SD: SD Oupiin 9004-BA09W01C00A - R1 Puede no conec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"
- board text added: "PRECAUCIÓN: NO PROGRAMAR CON LA ALIMENTACIÓN CONECTADA. ES ALTAMENTE RECOMENDABLE PROGRAMAR EL MICROCONTROLADOR ANTES DE CONECTARLO A ESTA PLACA. PUEDEN QUEMARSE LOS COMPONENTES."
- board text added: "TAUTOLOGICAL"
- board text added: "Valores: R1 = 0R (opcional) R2 = NO CONECTAR R3 = NO CONECTAR R4 = 1K8 R5 = 1K8 R6 = 1K8 R7 = 3K3 R8 = 3K3 R9 = 3K3 C1 = 1uF x 16V (polarizado) C2 = 100nF C3 = 100uF C4 = 330uF D1 = 1N5817 L1 = 330uH Choke PK0810"
Changed lines of the file:
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@@
     (links 118)
     (no_connects 0)
-    (area 86.435717 47.025 251.090857 162.7)
+    (area 13.799999 26.7 253.714284 194.025)
     (thickness 1.6)
-    (drawings 101)
+    (drawings 119)
     (tracks 658)
     (zones 0)
@@
   )
   (page A4)
+  (title_block
+    (title TAUTOLOGIAL)
+    (date 2018-10-30)
+    (rev A)
+    (company "UTN - FRBA")
+    (comment 1 https://github.com/ealegremendoza/proyecto_4to)
+    (comment 2 "Autores: Alegre M. E., Bautista L., Tarazona L.")
+    (comment 3 "Medidor de posición y velocidad de sujetos en movimiento")
+    (comment 4 "Sport Tracker")
+  )
   (layers
     (0 F.Cu signal)
@@
     (38 B.Mask user)
     (39 F.Mask user)
-    (40 Dwgs.User user hide)
+    (40 Dwgs.User user)
     (41 Cmts.User user)
     (42 Eco1.User user)
@@
       (effects (font (size 1 1) (thickness 0.25)))
     )
-    (fp_text value 330u (at 0 -6.46) (layer F.Fab)
+    (fp_text value 330u (at 0 -0.016) (layer F.Fab)
       (effects (font (size 1 1) (thickness 0.15)))
     )
@@
       (xy 2.823256 -3.900663)) (layer F.SilkS) (width 0.01))
   )
+  (gr_line (start 14 116) (end 21 104) (layer Cmts.User) (width 0.4))
+  (gr_line (start 28 116) (end 14 116) (layer Cmts.User) (width 0.4))
+  (gr_line (start 21 104) (end 28 116) (layer Cmts.User) (width 0.4))
+  (gr_text ! (at 21 111) (layer Cmts.User)
+    (effects (font (size 7 7) (thickness 1.25)))
+  )
+  (gr_text "PRECAUCIÓN:\nNO PROGRAMAR CON LA ALIMENTACIÓN \nCONECTADA.\nES ALTAMENTE RECOMENDABLE \nPROGRAMAR EL MICROCONTROLADOR \nANTES DE CONECTARLO A ESTA\nPLACA. \nPUEDEN QUEMARSE LOS COMPONENTES." (at 33 111) (layer Cmts.User)
+    (effects (font (size 2 2) (thickness 0.35)) (justify left))
+  )
+  (gr_text "PLACA BASE" (at 150 38) (layer Cmts.User)
+    (effects (font (size 1.5 1.5) (thickness 0.3)))
+  )
+  (gr_text TAUTOLOGICAL (at 150 30) (layer Cmts.User)
+    (effects (font (size 4 4) (thickness 1)))
+  )
+  (gr_text "Valores:\nR1 = 0R (opcional)\nR2 = NO CONECTAR\nR3 = NO CONECTAR\nR4 = 1K8\nR5 = 1K8\nR6 = 1K8\nR7 = 3K3\nR8 = 3K3\nR9 = 3K3\nC1 = 1uF x 16V (polarizado)\nC2 = 100nF\nC3 = 100uF\nC4 = 330uF\nD1 = 1N5817\nL1 = 330uH Choke PK0810" (at 220 100) (layer Cmts.User)
+    (effects (font (size 1.5 1.5) (thickness 0.3)) (justify left))
+  )
+  (gr_text 330uH (at 139 136) (layer F.Fab)
+    (effects (font (size 1 1) (thickness 0.15)))
+  )
+  (gr_text "IMPORTANTE.\n- El ARDUINO MEGA va conectado al revés, boca abajo.\nDeben soldarse tira de pines macho. En los 6 pines centrales de este deben \nsoldarse pines hembra.\n- Todos los resistores y C2 son 0805. |C1: CP_Tantalum_Case-A_EIA-3216-18. \nC4: CP_Elec_10x10.5. | C3:CP_Elec_6.3x5.3\n- Conector del GPS: JST_SH_SM06B-SRSS-TB_06x1.00mm_Angled.\n- Tarjeta SD: SD Oupiin 9004-BA09W01C00A\n- R1 Puede no conectarse. En este caso no afecta al funcionamiento del dispositivo\nya que es solo para redireccionamiento del mismo.\n- Debido a que no se hace uso de los pines PD (los inferiores), pueden usarse hasta \nla fecha las siguientes revisiones: B, C Y D. SIEMPRE QUE NO SE SUELDEN DICHOS \nPINES AL LPC Y/O A ESTA PLACA BASE.\n- Los 8 primeros pines del MPU9250 son perfectamente compatibles con el MPU6050.\n- Tener en cuenta que con la tarjeta SD montada sobre sale 11mm.\n- LM2575: TO-263-5_TabPin3\n- Ajustar todos los dispositivos con sus respectivos pasantes. Para eso se realizaron las perforaciones de 3.2mm.\nSe debe priorizar la estabilidad del dispositivo." (at 26 171) (layer Cmts.User)
+    (effects (font (size 1.5 1.5) (thickness 0.3)) (justify left))
+  )
+  (dimension 11 (width 0.3) (layer Dwgs.User)
+    (gr_text "11,000 mm" (at 177.770961 155.643756 90) (layer Dwgs.User)
+      (effects (font (size 1.5 1.5) (thickness 0.3)))
+    )
+    (feature1 (pts (xy 172.420962 150.143756) (xy 179.120961 150.143756)))
+    (feature2 (pts (xy 172.420962 161.143756) (xy 179.120961 161.143756)))
+    (crossbar (pts (xy 176.420961 161.143756) (xy 176.420961 150.143756)))
+    (arrow1a (pts (xy 176.420961 150.143756) (xy 177.007382 151.27026)))
+    (arrow1b (pts (xy 176.420961 150.143756) (xy 175.83454 151.27026)))
+    (arrow2a (pts (xy 176.420961 161.143756) (xy 177.007382 160.017252)))
+    (arrow2b (pts (xy 176.420961 161.143756) (xy 175.83454 160.017252)))
+  )
+  (dimension 5 (width 0.3) (layer Dwgs.User)
+    (gr_text "5,000 mm" (at 102.5 45.650001) (layer Dwgs.User)
+      (effects (font (size 1.5 1.5) (thickness 0.3)))
+    )
+    (feature1 (pts (xy 100 55) (xy 100 44.300001)))
+    (feature2 (pts (xy 105 55) (xy 105 44.300001)))
+    (crossbar (pts (xy 105 47.000001) (xy 100 47.000001)))
+    (arrow1a (pts (xy 100 47.000001) (xy 101.126504 46.41358)))
+    (arrow1b (pts (xy 100 47.000001) (xy 101.126504 47.586422)))
+    (arrow2a (pts (xy 105 47.000001) (xy 103.873496 46.41358)))
+    (arrow2b (pts (xy 105 47.000001) (xy 103.873496 47.586422)))
+  )
+  (dimension 5 (width 0.3) (layer Dwgs.User)
+    (gr_text "5,000 mm" (at 110.349999 52.5 90) (layer Dwgs.User)
+      (effects (font (size 1.5 1.5) (thickness 0.3)))
+    )
+    (feature1 (pts (xy 105 50) (xy 111.699999 50)))
+    (feature2 (pts (xy 105 55) (xy 111.699999 55)))
+    (crossbar (pts (xy 108.999999 55) (xy 108.999999 50)))
+    (arrow1a (pts (xy 108.999999 50) (xy 109.58642 51.126504)))
+    (arrow1b (pts (xy 108.999999 50) (xy 108.413578 51.126504)))
+    (arrow2a (pts (xy 108.999999 55) (xy 109.58642 53.873496)))
+    (arrow2b (pts (xy 108.999999 55) (xy 108.413578 53.873496)))
+  )
+  (dimension 5 (width 0.3) (layer Dwgs.User)
+    (gr_text "5,000 mm" (at 108.35 147.5 270) (layer Dwgs.User)
+      (effects (font (size 1.5 1.5) (thickness 0.3)))
+    )
+    (feature1 (pts (xy 105 150) (xy 109.7 150)))
+    (feature2 (pts (xy 105 145) (xy 109.7 145)))
+    (crossbar (pts (xy 107 145) (xy 107 150)))
+    (arrow1a (pts (xy 107 150) (xy 106.413579 148.873496)))
+    (arrow1b (pts (xy 107 150) (xy 107.586421 148.873496)))
+    (arrow2a (pts (xy 107 145) (xy 106.413579 146.126504)))
+    (arrow2b (pts (xy 107 145) (xy 107.586421 146.126504)))
+  )
+  (dimension 5 (width 0.3) (layer Dwgs.User)
+    (gr_text "5,000 mm" (at 102.5 141.650001) (layer Dwgs.User)
+      (effects (font (size 1.5 1.5) (thickness 0.3)))
+    )
+    (feature1 (pts (xy 100 145) (xy 100 140.300001)))
+    (feature2 (pts (xy 105 145) (xy 105 140.300001)))
+    (crossbar (pts (xy 105 143.000001) (xy 100 143.000001)))
+    (arrow1a (pts (xy 100 143.000001) (xy 101.126504 142.41358)))
+    (arrow1b (pts (xy 100 143.000001) (xy 101.126504 143.586422)))
+    (arrow2a (pts (xy 105 143.000001) (xy 103.873496 142.41358)))
+    (arrow2b (pts (xy 105 143.000001) (xy 103.873496 143.586422)))
+  )
+  (dimension 5.08 (width 0.3) (layer Dwgs.User)
+    (gr_text "5,080 mm" (at 126.48438 142.922) (layer Dwgs.User)
+      (effects (font (size 1.5 1.5) (thickness 0.3)))
+    )
+    (feature1 (pts (xy 129.02438 145.796) (xy 129.02438 141.572)))
+    (feature2 (pts (xy 123.94438 145.796) (xy 123.94438 141.572)))
+    (crossbar (pts (xy 123.94438 144.272) (xy 129.02438 144.272)))
+    (arrow1a (pts (xy 129.02438 144.272) (xy 127.897876 144.858421)))
+    (arrow1b (pts (xy 129.02438 144.272) (xy 127.897876 143.685579)))
+    (arrow2a (pts (xy 123.94438 144.272) (xy 125.070884 144.858421)))
+    (arrow2b (pts (xy 123.94438 144.272) (xy 125.070884 143.685579)))
+  )
+  (dimension 2.540011 (width 0.3) (layer Dwgs.User)
+    (gr_text "2,540 mm" (at 104.379813 85.674283 359.8281132) (layer Dwgs.User)
+      (effects (font (size 1.5 1.5) (thickness 0.3)))
+    )
+    (feature1 (pts (xy 105.66146 81.79562) (xy 105.645763 87.028087)))
+    (feature2 (pts (xy 103.12146 81.788) (xy 103.105763 87.020467)))
+    (crossbar (pts (xy 103.113863 84.320479) (xy 105.653863 84.328099)))
+    (arrow1a (pts (xy 105.653863 84.328099) (xy 104.525605 84.911138)))
+    (arrow1b (pts (xy 105.653863 84.328099) (xy 104.529124 83.738301)))
+    (arrow2a (pts (xy 103.113863 84.320479) (xy 104.238602 84.910277)))
+    (arrow2b (pts (xy 103.113863 84.320479) (xy 104.242121 83.73744)))
+  )
+  (dimension 2.540011 (width 0.3) (layer Dwgs.User)
+    (gr_text "2,540 mm" (at 139.517037 55.637213 89.82811318) (layer Dwgs.User)
+      (effects (font (size 1.5 1.5) (thickness 0.3)))
+    )
+    (feature1 (pts (xy 143.3957 56.91886) (xy 138.163233 56.903163)))
+    (feature2 (pts (xy 143.40332 54.37886) (xy 138.170853 54.363163)))
+    (crossbar (pts (xy 140.870841 54.371263) (xy 140.863221 56.911263)))
+    (arrow1a (pts (xy 140.863221 56.911263) (xy 140.280182 55.783005)))
+    (arrow1b (pts (xy 140.863221 56.911263) (xy 141.453019 55.786524)))
+    (arrow2a (pts (xy 140.870841 54.371263) (xy 140.281043 55.496002)))
+    (arrow2b (pts (xy 140.870841 54.371263) (xy 141.45388 55.499521)))
+  )
   (gr_text "Ailu  " (at 196.215 140.97) (layer B.Cu)
